File: kicad/µmotor-can.sch (KiCad schematic (older format))
At the start: 2 parts, among them U601 TCAN330

Commit message: update µC pinout, motor driver, CubeMX, add 3V3 regulator and temperature sensor
Connections:
- net +3V3 renamed 3V_IN
Other:
- moved on the sheet: C601
Changed lines of the file:
@@
 LIBS:drv8323s
 LIBS:FDMD82xx
+LIBS:ncp4623
+LIBS:TMP006
 LIBS:µmotor-cache
 EELAYER 25 0
@@
 $Descr A4 11693 8268
 encoding utf-8
-Sheet 6 6
+Sheet 4 6
 Title "µmotor - Micro Motor Controller"
 Date "2017-09-14"
@@
 $EndComp
 $Comp
-L +3V3 #PWR027
-U 1 1 59BAE85A
-P 5400 3350
-F 0 "#PWR027" H 5400 3200 50  0001 C CNN
-F 1 "+3V3" H 5400 3490 50  0000 C CNN
-F 2 "" H 5400 3350 50  0001 C CNN
-F 3 "" H 5400 3350 50  0001 C CNN
-	1    5400 3350
-	0    -1   -1   0
-$EndComp
-$Comp
 L GND #PWR028
 U 1 1 59BAE870
@@
 	5200 3250 5500 3250
 Wire Wire Line
-	5400 3350 5500 3350
+	4450 3350 5500 3350
 Wire Wire Line
 	4950 3450 5500 3450
@@
 L C C601
 U 1 1 59BAEA09
-P 5850 4300
-F 0 "C601" H 5875 4400 50  0000 L CNN
-F 1 "100n" H 5875 4200 50  0000 L CNN
-F 2 "Capacitors_SMD:C_0603" H 5888 4150 50  0001 C CNN
-F 3 "" H 5850 4300 50  0001 C CNN
-	1    5850 4300
-	1    0    0    -1
-$EndComp
-$Comp
-L +3V3 #PWR029
-U 1 1 59BAEB8F
-P 5850 4050
-F 0 "#PWR029" H 5850 3900 50  0001 C CNN
-F 1 "+3V3" H 5850 4190 50  0000 C CNN
-F 2 "" H 5850 4050 50  0001 C CNN
-F 3 "" H 5850 4050 50  0001 C CNN
-	1    5850 4050
+P 4500 3750
+F 0 "C601" H 4525 3850 50  0000 L CNN
+F 1 "100n" H 4525 3650 50  0000 L CNN
+F 2 "Capacitors_SMD:C_0603" H 4538 3600 50  0001 C CNN
+F 3 "" H 4500 3750 50  0001 C CNN
+	1    4500 3750
 	1    0    0    -1
 $EndComp
 Wire Wire Line
-	5850 4050 5850 4150
+	4500 3350 4500 3600
 $Comp
 L GND #PWR030
 U 1 1 59BAEBB1
-P 5850 4550
-F 0 "#PWR030" H 5850 4300 50  0001 C CNN
-F 1 "GND" H 5850 4400 50  0000 C CNN
-F 2 "" H 5850 4550 50  0001 C CNN
-F 3 "" H 5850 4550 50  0001 C CNN
-	1    5850 4550
+P 4500 4000
+F 0 "#PWR030" H 4500 3750 50  0001 C CNN
+F 1 "GND" H 4500 3850 50  0000 C CNN
+F 2 "" H 4500 4000 50  0001 C CNN
+F 3 "" H 4500 4000 50  0001 C CNN
+	1    4500 4000
 	1    0    0    -1
 $EndComp
 Wire Wire Line
-	5850 4550 5850 4450
+	4500 4000 4500 3900
+Text HLabel 4450 3350 0    60   Input ~ 0
+3V_IN
+Connection ~ 4500 3350
 $EndSCHEMATC

Commit message: layout: components placed
Parts:
- renumbered C601 to C401, U601 to U401
Connections:
- net 3V_IN renamed +3V3
Changed lines of the file:
@@
 LIBS:conn
 LIBS:linear
-LIBS:regul
-LIBS:74xx
-LIBS:cmos4000
-LIBS:adc-dac
-LIBS:memory
-LIBS:xilinx
-LIBS:microcontrollers
-LIBS:dsp
-LIBS:microchip
-LIBS:analog_switches
-LIBS:motorola
 LIBS:texas
-LIBS:intel
-LIBS:audio
 LIBS:interface
-LIBS:digital-audio
-LIBS:philips
-LIBS:display
-LIBS:cypress
-LIBS:siliconi
-LIBS:opto
-LIBS:atmel
 LIBS:contrib
 LIBS:valves
-LIBS:stm32
 LIBS:DRV8870
 LIBS:INA180A
@@
 LIBS:ncp4623
 LIBS:TMP006
+LIBS:stm32
 LIBS:µmotor-cache
 EELAYER 25 0
@@
 CAN_L
 $Comp
-L TCAN330 U601
+L TCAN330 U401
 U 1 1 59BAE765
 P 5950 3300
-F 0 "U601" H 5950 3600 60  0000 C CNN
+F 0 "U401" H 5950 3600 60  0000 C CNN
 F 1 "TCAN330" H 5950 3000 60  0000 C CNN
 F 2 "TO_SOT_Packages_SMD:SOT-23-8" H 5950 3250 60  0001 C CNN
@@
 $EndComp
 $Comp
-L GND #PWR028
+L GND #PWR023
 U 1 1 59BAE870
 P 5200 3250
-F 0 "#PWR028" H 5200 3000 50  0001 C CNN
+F 0 "#PWR023" H 5200 3000 50  0001 C CNN
 F 1 "GND" H 5200 3100 50  0000 C CNN
 F 2 "" H 5200 3250 50  0001 C CNN
@@
 	5200 3250 5500 3250
 Wire Wire Line
-	4450 3350 5500 3350
+	4400 3350 5500 3350
 Wire Wire Line
 	4950 3450 5500 3450
@@
 NoConn ~ 6400 3450
 $Comp
-L C C601
+L C C401
 U 1 1 59BAEA09
 P 4500 3750
-F 0 "C601" H 4525 3850 50  0000 L CNN
+F 0 "C401" H 4525 3850 50  0000 L CNN
 F 1 "100n" H 4525 3650 50  0000 L CNN
 F 2 "Capacitors_SMD:C_0603" H 4538 3600 50  0001 C CNN
@@
 	4500 3350 4500 3600
 $Comp
-L GND #PWR030
+L GND #PWR024
 U 1 1 59BAEBB1
 P 4500 4000
-F 0 "#PWR030" H 4500 3750 50  0001 C CNN
+F 0 "#PWR024" H 4500 3750 50  0001 C CNN
 F 1 "GND" H 4500 3850 50  0000 C CNN
 F 2 "" H 4500 4000 50  0001 C CNN
@@
 Wire Wire Line
 	4500 4000 4500 3900
-Text HLabel 4450 3350 0    60   Input ~ 0
-3V_IN
 Connection ~ 4500 3350
+$Comp
+L +3V3 #PWR025
+U 1 1 5A7765B1
+P 4400 3350
+F 0 "#PWR025" H 4400 3200 50  0001 C CNN
+F 1 "+3V3" H 4400 3490 50  0000 C CNN
+F 2 "" H 4400 3350 50  0001 C CNN
+F 3 "" H 4400 3350 50  0001 C CNN
+	1    4400 3350
+	0    -1   -1   0
+$EndComp
 $EndSCHEMATC
