File: kicad/µmotor.sch (KiCad schematic (older format))
At the start: 17 parts, among them J101 CAN+PWR, J102 U, J103 V, J104 W, J105 U, J106 V, J107 W, J108 5V, J109 3V3, J110 IO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

Commit message: layout: improvements
Parts:
- added J112: GND, Measurement_Point_Round-SMD-Pad_Smaller:Measurement_Point_Round-SMD-Pad_Smaller_0.75mm, symbol TEST_1P
Connections:
- net GND: now also J112.1
Changed lines of the file:
@@
 $EndComp
 $Comp
-L GND #PWR103
+L GND #PWR01
 U 1 1 59B9FFC7
 P 1250 4150
-F 0 "#PWR103" H 1250 3900 50  0001 C CNN
+F 0 "#PWR01" H 1250 3900 50  0001 C CNN
 F 1 "GND" H 1250 4000 50  0000 C CNN
 F 2 "" H 1250 4150 50  0001 C CNN
@@
 	1150 4350 2100 4350
 $Comp
-L +6V #PWR105
+L +6V #PWR02
 U 1 1 59BA046F
 P 1550 4050
-F 0 "#PWR105" H 1550 3900 50  0001 C CNN
+F 0 "#PWR02" H 1550 3900 50  0001 C CNN
 F 1 "+6V" V 1550 4250 50  0000 C CNN
 F 2 "" H 1550 4050 50  0001 C CNN
@@
 $EndComp
 $Comp
-L +24V #PWR104
+L +24V #PWR03
 U 1 1 59BA04C0
 P 1550 3950
-F 0 "#PWR104" H 1550 3800 50  0001 C CNN
+F 0 "#PWR03" H 1550 3800 50  0001 C CNN
 F 1 "+24V" V 1550 4150 50  0000 C CNN
 F 2 "" H 1550 3950 50  0001 C CNN
@@
 $EndComp
 $Comp
-L +6V #PWR101
+L +6V #PWR04
 U 1 1 5A768B01
 P 1000 5400
-F 0 "#PWR101" H 1000 5250 50  0001 C CNN
+F 0 "#PWR04" H 1000 5250 50  0001 C CNN
 F 1 "+6V" H 1000 5540 50  0000 C CNN
 F 2 "" H 1000 5400 50  0001 C CNN
@@
 	2850 5400 2850 5600
 $Comp
-L GND #PWR106
+L GND #PWR05
 U 1 1 5A769C21
 P 2050 6100
-F 0 "#PWR106" H 2050 5850 50  0001 C CNN
+F 0 "#PWR05" H 2050 5850 50  0001 C CNN
 F 1 "GND" H 2050 5950 50  0000 C CNN
 F 2 "" H 2050 6100 50  0001 C CNN
@@
 	7350 5200 8150 5200
 $Comp
-L +3V3 #PWR108
+L +3V3 #PWR06
 U 1 1 5A775FAA
 P 3150 5400
-F 0 "#PWR108" H 3150 5250 50  0001 C CNN
+F 0 "#PWR06" H 3150 5250 50  0001 C CNN
 F 1 "+3V3" H 3150 5540 50  0000 C CNN
 F 2 "" H 3150 5400 50  0001 C CNN
@@
 $EndComp
 $Comp
-L +6V #PWR102
+L +6V #PWR07
 U 1 1 5A77E4A3
 P 1000 6750
-F 0 "#PWR102" H 1000 6600 50  0001 C CNN
+F 0 "#PWR07" H 1000 6600 50  0001 C CNN
 F 1 "+6V" H 1000 6890 50  0000 C CNN
 F 2 "" H 1000 6750 50  0001 C CNN
@@
 	2850 6750 2850 6950
 $Comp
-L GND #PWR107
+L GND #PWR08
 U 1 1 5A77E4BD
 P 2050 7450
-F 0 "#PWR107" H 2050 7200 50  0001 C CNN
+F 0 "#PWR08" H 2050 7200 50  0001 C CNN
 F 1 "GND" H 2050 7300 50  0000 C CNN
 F 2 "" H 2050 7450 50  0001 C CNN
@@
 Connection ~ 2850 6750
 $Comp
-L +5V #PWR109
+L +5V #PWR09
 U 1 1 5A77E77B
 P 3150 6750
-F 0 "#PWR109" H 3150 6600 50  0001 C CNN
+F 0 "#PWR09" H 3150 6600 50  0001 C CNN
 F 1 "+5V" H 3150 6890 50  0000 C CNN
 F 2 "" H 3150 6750 50  0001 C CNN
@@
 $EndComp
 $Comp
-L +3V3 #PWR110
+L +3V3 #PWR010
 U 1 1 5A78722B
 P 3800 5450
-F 0 "#PWR110" H 3800 5300 50  0001 C CNN
+F 0 "#PWR010" H 3800 5300 50  0001 C CNN
 F 1 "+3V3" H 3800 5590 50  0000 C CNN
 F 2 "" H 3800 5450 50  0001 C CNN
@@
 $EndComp
 $Comp
-L GND #PWR111
+L GND #PWR011
 U 1 1 5A7873A5
 P 4000 5450
-F 0 "#PWR111" H 4000 5200 50  0001 C CNN
+F 0 "#PWR011" H 4000 5200 50  0001 C CNN
 F 1 "GND" H 4000 5300 50  0000 C CNN
 F 2 "" H 4000 5450 50  0001 C CNN
@@
 Wire Wire Line
 	4000 5450 4000 5350
+$Comp
+L TEST_1P J112
+U 1 1 5A7BE9B8
+P 4550 6850
+F 0 "J112" V 4550 7200 50  0000 C CNN
+F 1 "GND" H 4550 7050 50  0000 C CNN
+F 2 "Measurement_Point_Round-SMD-Pad_Smaller:Measurement_Point_Round-SMD-Pad_Smaller_0.75mm" H 4750 6850 50  0001 C CNN
+F 3 "" H 4750 6850 50  0001 C CNN
+	1    4550 6850
+	1    0    0    -1
+$EndComp
+$Comp
+L GND #PWR012
+U 1 1 5A7BE9BE
+P 4550 6950
+F 0 "#PWR012" H 4550 6700 50  0001 C CNN
+F 1 "GND" H 4550 6800 50  0000 C CNN
+F 2 "" H 4550 6950 50  0001 C CNN
+F 3 "" H 4550 6950 50  0001 C CNN
+	1    4550 6950
+	1    0    0    -1
+$EndComp
+Wire Wire Line
+	4550 6950 4550 6850
 $EndSCHEMATC
