File: kicad/macro-motor/macro-motor-can.sch (KiCad schematic (older format))
At the start: 2 parts, among them U401 TCAN330

Commit message: macro-motor: Finish dev board schematic
Parts:
- C401: symbol µmotor-rescue:C -> Device:C
Changed lines of the file:
@@
 EESchema Schematic File Version 4
-LIBS:µmotor-cache
+LIBS:macro-motor-cache
 EELAYER 26 0
 EELAYER END
@@
 $EndComp
 $Comp
-L power:GND #PWR031
+L power:GND #PWR0403
 U 1 1 59BAE870
 P 5200 3250
-F 0 "#PWR031" H 5200 3000 50  0001 C CNN
+F 0 "#PWR0403" H 5200 3000 50  0001 C CNN
 F 1 "GND" H 5200 3100 50  0000 C CNN
 F 2 "" H 5200 3250 50  0001 C CNN
@@
 NoConn ~ 6400 3450
 $Comp
-L µmotor-rescue:C C401
+L Device:C C?
 U 1 1 59BAEA09
 P 4500 3750
-AR Path="/59BAEA09" Ref="C401"  Part="1"
+AR Path="/59BAEA09" Ref="C?"  Part="1"
 AR Path="/59B9FE58/59BAEA09" Ref="C401"  Part="1"
 F 0 "C401" H 4525 3850 50  0000 L CNN
@@
 	4500 3350 4500 3600
 $Comp
-L power:GND #PWR032
+L power:GND #PWR0402
 U 1 1 59BAEBB1
 P 4500 4000
-F 0 "#PWR032" H 4500 3750 50  0001 C CNN
+F 0 "#PWR0402" H 4500 3750 50  0001 C CNN
 F 1 "GND" H 4500 3850 50  0000 C CNN
 F 2 "" H 4500 4000 50  0001 C CNN
@@
 Connection ~ 4500 3350
 $Comp
-L power:+3V3 #PWR033
+L power:+3V3 #PWR0401
 U 1 1 5A7765B1
 P 4400 3350
-F 0 "#PWR033" H 4400 3200 50  0001 C CNN
+F 0 "#PWR0401" H 4400 3200 50  0001 C CNN
 F 1 "+3V3" H 4400 3490 50  0000 C CNN
 F 2 "" H 4400 3350 50  0001 C CNN
