File: kicad/macro-motor/macro-motor.sch (KiCad schematic (older format))
At the start: 18 parts, among them J101 CAN+PWR, J102 U, J103 V, J104 W, J105 U, J106 V, J107 W, J108 5V, J109 Gpio, J111 GND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

Commit message: macro-motor: Finish dev board schematic
Parts:
- removed J102: U, Measurement_Points:Measurement_Point_Round-TH_Small, symbol µmotor-rescue:TEST_1P
- removed J103: V, Measurement_Points:Measurement_Point_Round-TH_Small, symbol µmotor-rescue:TEST_1P
- removed J104: W, Measurement_Points:Measurement_Point_Round-TH_Small, symbol µmotor-rescue:TEST_1P
- removed RN101: 1k, Local Footprints:EXB18V, symbol Device:R_Pack04
- removed RN102: 20k, Local Footprints:EXB18V, symbol Device:R_Pack04
- added J102: 3V3, Connector_Pin:Pin_D1.0mm_L10.0mm, symbol Connector:TestPoint
- added J109: Conn_01x03_Female, TerminalBlock_Phoenix:TerminalBlock_Phoenix_PT-1,5-3-3.5-H_1x03_P3.50mm_Horizontal, symbol Connector:Conn_01x03_Female
- added J110: HALL, Connector_PinHeader_2.54mm:PinHeader_1x05_P2.54mm_Vertical, symbol Connector:Conn_01x05_Male
- added J111: Fault, Connector_Pin:Pin_D1.0mm_L10.0mm, symbol Connector:TestPoint
- added R102, R103, R104: 1k, Resistor_SMD:R_0402_1005Metric, symbol Device:R
- added R105, R106, R107: 20k, Resistor_SMD:R_0402_1005Metric, symbol Device:R
- added R108: (10k), Resistor_SMD:R_0402_1005Metric, symbol Device:R
- C101: value 2µ2 16V -> 4µ7 16V; symbol µmotor-rescue:C -> Device:C
- C102: symbol µmotor-rescue:C -> Device:C
- C103: renamed from C104; symbol µmotor-rescue:C -> Device:C
- J101: footprint Pin_Headers:Pin_Header_Straight_1x05_Pitch2.54mm -> Connector_PinHeader_2.54mm:PinHeader_1x05_P2.54mm_Vertical; symbol µmotor-rescue:CONN_01X05 -> Connector:Conn_01x05_Male
- J103: renamed from J108; footprint Measurement_Point_Round-SMD-Pad_Smaller:Measurement_Point_Round-SMD-Pad_Smaller_0.75mm -> Connector_Pin:Pin_D1.0mm_L10.0mm; symbol µmotor-rescue:TEST_1P -> Connector:TestPoint
- J104: renamed from J111; footprint Measurement_Point_Round-SMD-Pad_Smaller:Measurement_Point_Round-SMD-Pad_Smaller_0.75mm -> Connector_Pin:Pin_D1.0mm_L10.0mm; symbol µmotor-rescue:TEST_1P -> Connector:TestPoint
- J105: renamed from J109; footprint Measurement_Point_Round-SMD-Pad_Smaller:Measurement_Point_Round-SMD-Pad_Smaller_0.75mm -> Connector_Pin:Pin_D1.0mm_L10.0mm; symbol µmotor-rescue:TEST_1P -> Connector:TestPoint
- J106: renamed from J105; footprint Measurement_Point_Round-SMD-Pad_Smaller:Measurement_Point_Round-SMD-Pad_Smaller_0.75mm -> Connector_Pin:Pin_D1.0mm_L10.0mm; symbol µmotor-rescue:TEST_1P -> Connector:TestPoint
- J107: renamed from J106; footprint Measurement_Point_Round-SMD-Pad_Smaller:Measurement_Point_Round-SMD-Pad_Smaller_0.75mm -> Connector_Pin:Pin_D1.0mm_L10.0mm; symbol µmotor-rescue:TEST_1P -> Connector:TestPoint
- J108: renamed from J107; footprint Measurement_Point_Round-SMD-Pad_Smaller:Measurement_Point_Round-SMD-Pad_Smaller_0.75mm -> Connector_Pin:Pin_D1.0mm_L10.0mm; symbol µmotor-rescue:TEST_1P -> Connector:TestPoint
Connections:
- wire segments 97 -> 112
- no-connect marks 6 -> 2
