File: kicad/macro-motor/macro-motor-microcontroller.sch (KiCad schematic (older format))
At the start: 15 parts, among them J601 GND, J602 SWCLK, J603 SWDIO, J604 TX, U601 STM32L433C(B-C)Ux_u

Commit message: macro-motor: Finish dev board schematic
Parts:
- removed J601: GND, Measurement_Point_Round-SMD-Pad_Smaller:Measurement_Point_Round-SMD-Pad_Smaller_0.75mm, symbol µmotor-rescue:TEST_1P
- removed J602: SWCLK, Measurement_Point_Round-SMD-Pad_Smaller:Measurement_Point_Round-SMD-Pad_Smaller_0.5mm, symbol µmotor-rescue:TEST_1P
- removed J603: SWDIO, Measurement_Point_Round-SMD-Pad_Smaller:Measurement_Point_Round-SMD-Pad_Smaller_0.5mm, symbol µmotor-rescue:TEST_1P
- removed J604: TX, Measurement_Point_Round-SMD-Pad_Smaller:Measurement_Point_Round-SMD-Pad_Smaller_0.5mm, symbol µmotor-rescue:TEST_1P
- removed RN601: 10k, Local Footprints:EXB18V, symbol Device:R_Pack04
- added J601: SWD, Connector_PinHeader_2.54mm:PinHeader_1x03_P2.54mm_Vertical, symbol Connector:Conn_01x03_Male
- added J604: UART, Connector_PinHeader_2.54mm:PinHeader_1x03_P2.54mm_Vertical, symbol Connector:Conn_01x03_Male
- added J605: OP_INM, Connector_Pin:Pin_D1.0mm_L10.0mm, symbol Connector:TestPoint
- added J606: OP_OUT, Connector_Pin:Pin_D1.0mm_L10.0mm, symbol Connector:TestPoint
- added J607: PA0, Connector_Pin:Pin_D1.0mm_L10.0mm, symbol Connector:TestPoint
- added J608: PH1, Connector_Pin:Pin_D1.0mm_L10.0mm, symbol Connector:TestPoint
- added J609: PH0, Connector_Pin:Pin_D1.0mm_L10.0mm, symbol Connector:TestPoint
- added R605, R606, R607, R608: 10k, Resistor_SMD:R_0402_1005Metric, symbol Device:R
- C601: renamed from C603; symbol µmotor-rescue:C -> Device:C
- C602: renamed from C601; symbol µmotor-rescue:C -> Device:C
- C603: renamed from C602; symbol µmotor-rescue:C -> Device:C
- D601, D602: symbol µmotor-rescue:LED -> Device:LED
- R601, R602: symbol µmotor-rescue:R -> Device:R
- U601: footprint Package_DFN_QFN:QFN-48-1EP_7x7mm_P0.5mm_EP5.3x5.3mm -> Package_DFN_QFN:QFN-48-1EP_7x7mm_P0.5mm_EP5.6x5.6mm
Connections:
- net labels added: PA0, PH0, PH1
- wire segments 97 -> 103
- no-connect marks 0 -> 1
Other:
- note removed: "SWD"
- note removed: "UART"

Commit message: macro-motor: PCB Layout
Parts:
- C601: value 10n??? -> 100n
Changed lines of the file:
@@
 AR Path="/59B9FC4A/5A7A4571" Ref="C601"  Part="1"
 F 0 "C601" H 1475 7150 50  0000 L CNN
-F 1 "10n???" H 1475 6950 50  0000 L CNN
+F 1 "100n" H 1475 6950 50  0000 L CNN
 F 2 "Capacitor_SMD:C_0402_1005Metric" H 1488 6900 50  0001 C CNN
 F 3 "" H 1450 7050 50  0001 C CNN
