File: kicad/macro-motor/macro-motor-temp-sensor.sch (KiCad schematic (older format))
At the start: 7 parts, among them J501 SCL, J502 SDA, J503 3V3, J504 GND, U501 TMP006

Commit message: macro-motor: Finish dev board schematic
Parts:
- J501, J502, J503, J504: footprint Measurement_Point_Round-SMD-Pad_Smaller:Measurement_Point_Round-SMD-Pad_Smaller_0.75mm -> Connector_Pin:Pin_D1.0mm_L10.0mm; symbol µmotor-rescue:TEST_1P -> Connector:TestPoint
- R501, R502: symbol µmotor-rescue:R -> Device:R
Changed lines of the file:
@@
 EESchema Schematic File Version 4
-LIBS:µmotor-cache
+LIBS:macro-motor-cache
 EELAYER 26 0
 EELAYER END
@@
 NoConn ~ 4550 2200
 $Comp
-L power:GND #PWR034
+L power:GND #PWR0503
 U 1 1 5A76B49A
 P 4650 2500
-F 0 "#PWR034" H 4650 2250 50  0001 C CNN
+F 0 "#PWR0503" H 4650 2250 50  0001 C CNN
 F 1 "GND" H 4650 2350 50  0000 C CNN
 F 2 "" H 4650 2500 50  0001 C CNN
@@
 Connection ~ 4650 2400
 $Comp
-L power:GND #PWR035
+L power:GND #PWR0502
 U 1 1 5A76B4B9
 P 3550 2400
-F 0 "#PWR035" H 3550 2150 50  0001 C CNN
+F 0 "#PWR0502" H 3550 2150 50  0001 C CNN
 F 1 "GND" H 3550 2250 50  0000 C CNN
 F 2 "" H 3550 2400 50  0001 C CNN
@@
 Connection ~ 3550 2300
 $Comp
-L power:+3V3 #PWR036
+L power:+3V3 #PWR0501
 U 1 1 5A76B4E0
 P 3550 2000
-F 0 "#PWR036" H 3550 1850 50  0001 C CNN
+F 0 "#PWR0501" H 3550 1850 50  0001 C CNN
 F 1 "+3V3" H 3550 2140 50  0000 C CNN
 F 2 "" H 3550 2000 50  0001 C CNN
@@
 	4550 2100 4850 2100
 $Comp
-L µmotor-rescue:TEST_1P J501
+L Connector:TestPoint J?
 U 1 1 5A76B941
 P 5200 1900
-AR Path="/5A76B941" Ref="J501"  Part="1"
+AR Path="/5A76B941" Ref="J?"  Part="1"
 AR Path="/59BA5FB5/5A76B941" Ref="J501"  Part="1"
 F 0 "J501" H 5200 2170 50  0000 C CNN
 F 1 "SCL" H 5200 2100 50  0000 C CNN
-F 2 "Measurement_Point_Round-SMD-Pad_Smaller:Measurement_Point_Round-SMD-Pad_Smaller_0.75mm" H 5400 1900 50  0001 C CNN
+F 2 "Connector_Pin:Pin_D1.0mm_L10.0mm" H 5400 1900 50  0001 C CNN
 F 3 "" H 5400 1900 50  0001 C CNN
 	1    5200 1900
@@
 $EndComp
 $Comp
-L µmotor-rescue:TEST_1P J502
+L Connector:TestPoint J?
 U 1 1 5A76B97E
 P 5200 2200
-AR Path="/5A76B97E" Ref="J502"  Part="1"
+AR Path="/5A76B97E" Ref="J?"  Part="1"
 AR Path="/59BA5FB5/5A76B97E" Ref="J502"  Part="1"
 F 0 "J502" H 5200 2470 50  0000 C CNN
 F 1 "SDA" H 5200 2400 50  0000 C CNN
-F 2 "Measurement_Point_Round-SMD-Pad_Smaller:Measurement_Point_Round-SMD-Pad_Smaller_0.75mm" H 5400 2200 50  0001 C CNN
+F 2 "Connector_Pin:Pin_D1.0mm_L10.0mm" H 5400 2200 50  0001 C CNN
 F 3 "" H 5400 2200 50  0001 C CNN
 	1    5200 2200
@@
 Connection ~ 5200 2000
 $Comp
-L µmotor-rescue:TEST_1P J503
+L Connector:TestPoint J?
 U 1 1 5A77F3B3
 P 6450 2100
-AR Path="/5A77F3B3" Ref="J503"  Part="1"
+AR Path="/5A77F3B3" Ref="J?"  Part="1"
 AR Path="/59BA5FB5/5A77F3B3" Ref="J503"  Part="1"
 F 0 "J503" H 6450 2370 50  0000 C CNN
 F 1 "3V3" H 6450 2300 50  0000 C CNN
-F 2 "Measurement_Point_Round-SMD-Pad_Smaller:Measurement_Point_Round-SMD-Pad_Smaller_0.75mm" H 6650 2100 50  0001 C CNN
+F 2 "Connector_Pin:Pin_D1.0mm_L10.0mm" H 6650 2100 50  0001 C CNN
 F 3 "" H 6650 2100 50  0001 C CNN
 	1    6450 2100
@@
 $EndComp
 $Comp
-L µmotor-rescue:TEST_1P J504
+L Connector:TestPoint J?
 U 1 1 5A77F3FB
 P 6700 2100
-AR Path="/5A77F3FB" Ref="J504"  Part="1"
+AR Path="/5A77F3FB" Ref="J?"  Part="1"
 AR Path="/59BA5FB5/5A77F3FB" Ref="J504"  Part="1"
 F 0 "J504" H 6700 2370 50  0000 C CNN
 F 1 "GND" H 6700 2300 50  0000 C CNN
-F 2 "Measurement_Point_Round-SMD-Pad_Smaller:Measurement_Point_Round-SMD-Pad_Smaller_0.75mm" H 6900 2100 50  0001 C CNN
+F 2 "Connector_Pin:Pin_D1.0mm_L10.0mm" H 6900 2100 50  0001 C CNN
 F 3 "" H 6900 2100 50  0001 C CNN
 	1    6700 2100
@@
 $EndComp
 $Comp
-L power:GND #PWR037
+L power:GND #PWR0506
 U 1 1 5A77F465
 P 6700 2200
-F 0 "#PWR037" H 6700 1950 50  0001 C CNN
+F 0 "#PWR0506" H 6700 1950 50  0001 C CNN
 F 1 "GND" H 6700 2050 50  0000 C CNN
 F 2 "" H 6700 2200 50  0001 C CNN
@@
 	6700 2200 6700 2100
 $Comp
-L power:+3V3 #PWR038
+L power:+3V3 #PWR0505
 U 1 1 5A77F497
 P 6450 2200
-F 0 "#PWR038" H 6450 2050 50  0001 C CNN
+F 0 "#PWR0505" H 6450 2050 50  0001 C CNN
 F 1 "+3V3" H 6450 2340 50  0000 C CNN
 F 2 "" H 6450 2200 50  0001 C CNN
@@
 	6450 2200 6450 2100
 $Comp
-L µmotor-rescue:R R501
+L Device:R R?
 U 1 1 5B469BD6
 P 4650 1600
-AR Path="/5B469BD6" Ref="R501"  Part="1"
+AR Path="/5B469BD6" Ref="R?"  Part="1"
 AR Path="/59BA5FB5/5B469BD6" Ref="R501"  Part="1"
 F 0 "R501" V 4730 1600 50  0000 C CNN
@@
 $EndComp
 $Comp
-L µmotor-rescue:R R502
+L Device:R R?
 U 1 1 5B469C77
 P 4850 1600
-AR Path="/5B469C77" Ref="R502"  Part="1"
+AR Path="/5B469C77" Ref="R?"  Part="1"
 AR Path="/59BA5FB5/5B469C77" Ref="R502"  Part="1"
 F 0 "R502" V 4930 1600 50  0000 C CNN
@@
 Connection ~ 4850 2100
 $Comp
-L power:+3V3 #PWR039
+L power:+3V3 #PWR0504
 U 1 1 5B469D07
 P 4750 1250
-F 0 "#PWR039" H 4750 1100 50  0001 C CNN
+F 0 "#PWR0504" H 4750 1100 50  0001 C CNN
 F 1 "+3V3" H 4750 1390 50  0000 C CNN
 F 2 "" H 4750 1250 50  0001 C CNN

Commit message: macro-motor: PCB Layout
Parts:
- added C501: 100n, Capacitor_SMD:C_0402_1005Metric, symbol Device:C
Connections:
- wire segments 27 -> 33
Changed lines of the file:
@@
 L power:GND #PWR0502
 U 1 1 5A76B4B9
-P 3550 2400
-F 0 "#PWR0502" H 3550 2150 50  0001 C CNN
-F 1 "GND" H 3550 2250 50  0000 C CNN
-F 2 "" H 3550 2400 50  0001 C CNN
-F 3 "" H 3550 2400 50  0001 C CNN
-	1    3550 2400
+P 3550 2500
+F 0 "#PWR0502" H 3550 2250 50  0001 C CNN
+F 1 "GND" H 3550 2350 50  0000 C CNN
+F 2 "" H 3550 2500 50  0001 C CNN
+F 3 "" H 3550 2500 50  0001 C CNN
+	1    3550 2500
 	1    0    0    -1
 $EndComp
@@
 L power:+3V3 #PWR0501
 U 1 1 5A76B4E0
-P 3550 2000
-F 0 "#PWR0501" H 3550 1850 50  0001 C CNN
-F 1 "+3V3" H 3550 2140 50  0000 C CNN
-F 2 "" H 3550 2000 50  0001 C CNN
-F 3 "" H 3550 2000 50  0001 C CNN
-	1    3550 2000
-	1    0    0    -1
-$EndComp
-Wire Wire Line
-	3550 2000 3550 2100
+P 3550 1800
+F 0 "#PWR0501" H 3550 1650 50  0001 C CNN
+F 1 "+3V3" H 3550 1940 50  0000 C CNN
+F 2 "" H 3550 1800 50  0001 C CNN
+F 3 "" H 3550 1800 50  0001 C CNN
+	1    3550 1800
+	1    0    0    -1
+$EndComp
 Wire Wire Line
 	3550 2100 3650 2100
@@
 Wire Wire Line
 	4750 1350 4850 1350
+$Comp
+L Device:C C501
+U 1 1 5BA90BBE
+P 3200 2150
+F 0 "C501" H 3315 2196 50  0000 L CNN
+F 1 "100n" H 3315 2105 50  0000 L CNN
+F 2 "Capacitor_SMD:C_0402_1005Metric" H 3238 2000 50  0001 C CNN
+F 3 "~" H 3200 2150 50  0001 C CNN
+	1    3200 2150
+	1    0    0    -1
+$EndComp
+Wire Wire Line
+	3550 1800 3550 1900
+Wire Wire Line
+	3550 1900 3200 1900
+Wire Wire Line
+	3200 1900 3200 2000
+Connection ~ 3550 1900
+Wire Wire Line
+	3550 1900 3550 2100
+Wire Wire Line
+	3200 2300 3200 2400
+Wire Wire Line
+	3200 2400 3550 2400
+Connection ~ 3550 2400
+Wire Wire Line
+	3550 2500 3550 2400
 $EndSCHEMATC
