File: kicad/macro-motor/macro-motor-encoder.sch (KiCad schematic (older format))
At the start: 9 parts, among them J201 A, J202 B, J204 GND, U201 AS5045B

Commit message: macro-motor: Finish dev board schematic
Parts:
- removed C201: 100n, Capacitor_SMD:C_0402_1005Metric, symbol µmotor-rescue:C
- removed D201: Red, LED_SMD:LED_0402_1005Metric, symbol µmotor-rescue:LED
- removed D202: Yellow, LED_SMD:LED_0402_1005Metric, symbol µmotor-rescue:LED
- removed J204: GND, Measurement_Point_Round-SMD-Pad_Smaller:Measurement_Point_Round-SMD-Pad_Smaller_0.75mm, symbol µmotor-rescue:TEST_1P
- removed R201, R202: 1k, Resistor_SMD:R_0402_1005Metric, symbol µmotor-rescue:R
- removed U201: AS5045B, Package_SO:SSOP-16_4.4x5.2mm_P0.65mm, symbol AS5045B:AS5045B
- added C201: 100n, Capacitor_SMD:C_0402_1005Metric, symbol Device:C
- added C202, C203, C204, C205: (2n7), Capacitor_SMD:C_0402_1005Metric, symbol Device:C
- added J204: Encoder, Connector_PinHeader_2.54mm:PinHeader_1x06_P2.54mm_Vertical, symbol Connector:Conn_01x06_Male
- added R203, R204, R205, R206: 47k, Resistor_SMD:R_0402_1005Metric, symbol Device:R
- added RN201: (2k7), local-lib:EXB18V, symbol Device:R_Pack04
- added RN202: (100), local-lib:EXB18V, symbol Device:R_Pack04
- added U202: UA9637, Package_SO:SOIC-8_3.9x4.9mm_P1.27mm, symbol Interface_LineDriver:UA9637
- J202: footprint Measurement_Point_Round-SMD-Pad_Smaller:Measurement_Point_Round-SMD-Pad_Smaller_0.75mm -> Connector_Pin:Pin_D1.0mm_L10.0mm; symbol µmotor-rescue:TEST_1P -> Connector:TestPoint
- J203: renamed from J201; footprint Measurement_Point_Round-SMD-Pad_Smaller:Measurement_Point_Round-SMD-Pad_Smaller_0.75mm -> Connector_Pin:Pin_D1.0mm_L10.0mm; symbol µmotor-rescue:TEST_1P -> Connector:TestPoint
Connections:
- net labels added: +5V
- wire segments 31 -> 77
- no-connect marks 5 -> 0
Other:
- note added: "5V/2 high-impedance voltage divider\n(If pins 1 and 6 are not connected)"
- note added: "TODO: RC Filter\n"

Commit message: macro-motor: PCB Layout
Other:
- note removed: "TODO: RC Filter\n"
Changed lines of the file:
@@
 Wire Wire Line
 	2900 4250 2900 4350
-Text Notes 3200 3950 0    50   ~ 0
-TODO: RC Filter\n
 Wire Wire Line
 	7050 3750 7150 3750

Commit message: macro-motor: Minor fixes
Parts:
- removed U202: UA9637, Package_SO:SOIC-8_3.9x4.9mm_P1.27mm, symbol Interface_LineDriver:UA9637
- added C206: 100n, Capacitor_SMD:C_0402_1005Metric, symbol Device:C
- added U201, U202: ISL3280E, Package_TO_SOT_SMD:SOT-23-5, symbol ISL3280E:ISL3280E
Connections:
- wire segments 77 -> 79
Changed lines of the file:
@@
 	3500 3150 3500 3250
-$Comp
-L Interface_LineDriver:UA9637 U202
-U 1 1 5BAB101B
-P 6550 3750
-F 0 "U202" H 6750 3550 50  0000 C CNN
-F 1 "UA9637" H 6750 3650 50  0000 C CNN
-F 2 "Package_SO:SOIC-8_3.9x4.9mm_P1.27mm" H 6550 3350 50  0001 C CNN
-F 3 "http://pdf.datasheetcatalog.com/datasheets2/28/284473_1.pdf" H 6550 3750 50  0001 C CNN
-	1    6550 3750
-	1    0    0    -1
-$EndComp
-$Comp
-L Interface_LineDriver:UA9637 U202
-U 2 1 5BAB10F0
-P 6250 4500
-F 0 "U202" H 6791 4546 50  0000 L CNN
-F 1 "UA9637" H 6791 4455 50  0000 L CNN
-F 2 "Package_SO:SOIC-8_3.9x4.9mm_P1.27mm" H 6250 4100 50  0001 C CNN
-F 3 "http://pdf.datasheetcatalog.com/datasheets2/28/284473_1.pdf" H 6250 4500 50  0001 C CNN
-	2    6250 4500
-	1    0    0    -1
-$EndComp
 $Comp
 L power:GND #PWR0121
@@
 L Device:C C201
 U 1 1 5BAAE514
-P 2900 4500
-F 0 "C201" H 3015 4546 50  0000 L CNN
-F 1 "100n" H 3015 4455 50  0000 L CNN
-F 2 "Capacitor_SMD:C_0402_1005Metric" H 2938 4350 50  0001 C CNN
-F 3 "~" H 2900 4500 50  0001 C CNN
-	1    2900 4500
+P 6850 5550
+F 0 "C201" H 6965 5596 50  0000 L CNN
+F 1 "100n" H 6965 5505 50  0000 L CNN
+F 2 "Capacitor_SMD:C_0402_1005Metric" H 6888 5400 50  0001 C CNN
+F 3 "~" H 6850 5550 50  0001 C CNN
+	1    6850 5550
 	1    0    0    -1
 $EndComp
@@
 L power:GND #PWR0126
 U 1 1 5BAAE64D
-P 2900 4750
-F 0 "#PWR0126" H 2900 4500 50  0001 C CNN
-F 1 "GND" H 2905 4577 50  0000 C CNN
-F 2 "" H 2900 4750 50  0001 C CNN
-F 3 "" H 2900 4750 50  0001 C CNN
-	1    2900 4750
-	1    0    0    -1
-$EndComp
-Wire Wire Line
-	2900 4750 2900 4650
+P 6850 5800
+F 0 "#PWR0126" H 6850 5550 50  0001 C CNN
+F 1 "GND" H 6855 5627 50  0000 C CNN
+F 2 "" H 6850 5800 50  0001 C CNN
+F 3 "" H 6850 5800 50  0001 C CNN
+	1    6850 5800
+	1    0    0    -1
+$EndComp
+Wire Wire Line
+	6850 5800 6850 5700
 $Comp
 L power:+3V3 #PWR0127
 U 1 1 5BAAEDB3
-P 2900 4250
-F 0 "#PWR0127" H 2900 4100 50  0001 C CNN
-F 1 "+3V3" H 2915 4423 50  0000 C CNN
-F 2 "" H 2900 4250 50  0001 C CNN
-F 3 "" H 2900 4250 50  0001 C CNN
-	1    2900 4250
-	1    0    0    -1
-$EndComp
-Wire Wire Line
-	2900 4250 2900 4350
-Wire Wire Line
-	7050 3750 7150 3750
-Wire Wire Line
-	7150 4500 6750 4500
+P 6850 5300
+F 0 "#PWR0127" H 6850 5150 50  0001 C CNN
+F 1 "+3V3" H 6865 5473 50  0000 C CNN
+F 2 "" H 6850 5300 50  0001 C CNN
+F 3 "" H 6850 5300 50  0001 C CNN
+	1    6850 5300
+	1    0    0    -1
+$EndComp
+Wire Wire Line
+	6850 5300 6850 5400
 $Comp
 L Device:R_Pack04 RN201
@@
 	5700 4200 5700 4400
 Wire Wire Line
-	5700 4400 5750 4400
-Wire Wire Line
 	5600 4300 5600 4600
 Wire Wire Line
-	5600 4600 5750 4600
-Wire Wire Line
 	5950 4100 5950 3850
-Wire Wire Line
-	5950 3850 6050 3850
-Wire Wire Line
-	6050 3650 5850 3650
 Wire Wire Line
 	5850 3650 5850 4000
@@
 Wire Wire Line
 	5150 4200 5700 4200
+$Comp
+L ISL3280E:ISL3280E U202
+U 1 1 5BAB59EB
+P 6600 3750
+F 0 "U202" H 6991 3796 50  0000 L CNN
+F 1 "ISL3280E" H 6991 3705 50  0000 L CNN
+F 2 "Package_TO_SOT_SMD:SOT-23-5" H 6600 3750 50  0001 C CNN
+F 3 "" H 6600 3750 50  0001 C CNN
+	1    6600 3750
+	1    0    0    -1
+$EndComp
+$Comp
+L ISL3280E:ISL3280E U201
+U 1 1 5BAB5CB0
+P 6300 4500
+F 0 "U201" H 6691 4546 50  0000 L CNN
+F 1 "ISL3280E" H 6691 4455 50  0000 L CNN
+F 2 "Package_TO_SOT_SMD:SOT-23-5" H 6300 4500 50  0001 C CNN
+F 3 "" H 6300 4500 50  0001 C CNN
+	1    6300 4500
+	1    0    0    -1
+$EndComp
+Wire Wire Line
+	6650 4500 7150 4500
+Wire Wire Line
+	5600 4600 5950 4600
+Wire Wire Line
+	5700 4400 5950 4400
+Wire Wire Line
+	5950 3850 6250 3850
+Wire Wire Line
+	5850 3650 6250 3650
+Wire Wire Line
+	6950 3750 7150 3750
+$Comp
+L Device:C C206
+U 1 1 5BAC18E2
+P 7300 5550
+F 0 "C206" H 7415 5596 50  0000 L CNN
+F 1 "100n" H 7415 5505 50  0000 L CNN
+F 2 "Capacitor_SMD:C_0402_1005Metric" H 7338 5400 50  0001 C CNN
+F 3 "~" H 7300 5550 50  0001 C CNN
+	1    7300 5550
+	1    0    0    -1
+$EndComp
+$Comp
+L power:GND #PWR0134
+U 1 1 5BAC18E8
+P 7300 5800
+F 0 "#PWR0134" H 7300 5550 50  0001 C CNN
+F 1 "GND" H 7305 5627 50  0000 C CNN
+F 2 "" H 7300 5800 50  0001 C CNN
+F 3 "" H 7300 5800 50  0001 C CNN
+	1    7300 5800
+	1    0    0    -1
+$EndComp
+Wire Wire Line
+	7300 5800 7300 5700
+$Comp
+L power:+3V3 #PWR0135
+U 1 1 5BAC18EF
+P 7300 5300
+F 0 "#PWR0135" H 7300 5150 50  0001 C CNN
+F 1 "+3V3" H 7315 5473 50  0000 C CNN
+F 2 "" H 7300 5300 50  0001 C CNN
+F 3 "" H 7300 5300 50  0001 C CNN
+	1    7300 5300
+	1    0    0    -1
+$EndComp
+Wire Wire Line
+	7300 5300 7300 5400
 $EndSCHEMATC
