File: kicad/macro-motor/macro-motor-motor-driver.sch (KiCad schematic (older format))
At the start: 12 parts, among them Q301 FDMD82xx, Q302 FDMD82xx, Q303 FDMD82xx, U301 DRV8323S

Commit message: macro-motor: Finish dev board schematic
Parts:
- added C301: >10µ 35V, Capacitor_THT:CP_Radial_D8.0mm_P3.50mm, symbol Device:CP
- added J301: A, Connector_PinHeader_2.54mm:PinHeader_1x02_P2.54mm_Vertical, symbol Connector:Conn_01x02_Female
- added J302: B, Connector_PinHeader_2.54mm:PinHeader_1x02_P2.54mm_Vertical, symbol Connector:Conn_01x02_Female
- added J303: C, Connector_PinHeader_2.54mm:PinHeader_1x02_P2.54mm_Vertical, symbol Connector:Conn_01x02_Female
- added JP301: SPC, Jumper:SolderJumper-2_P1.3mm_Open_RoundedPad1.0x1.5mm, symbol Jumper:SolderJumper_2_Open
- added JP302: SPB, Jumper:SolderJumper-2_P1.3mm_Open_RoundedPad1.0x1.5mm, symbol Jumper:SolderJumper_2_Open
- added JP303: SPA, Jumper:SolderJumper-2_P1.3mm_Open_RoundedPad1.0x1.5mm, symbol Jumper:SolderJumper_2_Open
- added R302, R303, R304: 5m, Resistor_SMD:R_0805_2012Metric, symbol Device:R
- added TP303, TP304: UP, Connector_Pin:Pin_D1.0mm_L10.0mm, symbol Connector:TestPoint
- added TP305: VP, Connector_Pin:Pin_D1.0mm_L10.0mm, symbol Connector:TestPoint
- added TP306: VN, Connector_Pin:Pin_D1.0mm_L10.0mm, symbol Connector:TestPoint
- added TP307: WP, Connector_Pin:Pin_D1.0mm_L10.0mm, symbol Connector:TestPoint
- added TP308: WN, Connector_Pin:Pin_D1.0mm_L10.0mm, symbol Connector:TestPoint
- added TP309: MOSI, Connector_Pin:Pin_D1.0mm_L10.0mm, symbol Connector:TestPoint
- added TP310: MISO, Connector_Pin:Pin_D1.0mm_L10.0mm, symbol Connector:TestPoint
- added TP311: SCK, Connector_Pin:Pin_D1.0mm_L10.0mm, symbol Connector:TestPoint
- added TP312: ~CS, Connector_Pin:Pin_D1.0mm_L10.0mm, symbol Connector:TestPoint
- added TP313, TP322: W, Connector_Pin:Pin_D1.0mm_L10.0mm, symbol Connector:TestPoint
- added TP314, TP323: V, Connector_Pin:Pin_D1.0mm_L10.0mm, symbol Connector:TestPoint
- added TP315, TP324: U, Connector_Pin:Pin_D1.0mm_L10.0mm, symbol Connector:TestPoint
- added TP316: GH_U, Connector_Pin:Pin_D1.0mm_L10.0mm, symbol Connector:TestPoint
- added TP317: GL_U, Connector_Pin:Pin_D1.0mm_L10.0mm, symbol Connector:TestPoint
- added TP318: GH_W, Connector_Pin:Pin_D1.0mm_L10.0mm, symbol Connector:TestPoint
- added TP319: GL_W, Connector_Pin:Pin_D1.0mm_L10.0mm, symbol Connector:TestPoint
- added TP320: GH_V, Connector_Pin:Pin_D1.0mm_L10.0mm, symbol Connector:TestPoint
- added TP321: GL_V, Connector_Pin:Pin_D1.0mm_L10.0mm, symbol Connector:TestPoint
- C302: symbol µmotor-rescue:C -> Device:C
- C303: renamed from C306; symbol µmotor-rescue:C -> Device:C
- C304: renamed from C303; symbol µmotor-rescue:C -> Device:C
- C305: renamed from C304; symbol µmotor-rescue:C -> Device:C
- C306: renamed from C305; symbol µmotor-rescue:C -> Device:C
- R301: renamed from R304; symbol µmotor-rescue:R -> Device:R
- TP301, TP302: footprint TestPoint:TestPoint_THTPad_D1.0mm_Drill0.5mm -> Connector_Pin:Pin_D1.0mm_L10.0mm
Connections:
- wire segments 159 -> 252
- no-connect marks 4 -> 1
Other:
- note added: "Optional:\nSHx pins will be used for SPx\n(DRV8323S CSA_FET bit)"
- note removed: "SHx pins will be used for SPx\n(DRV8323S CSA_FET bit)"

Commit message: macro-motor: Minor fixes
Connections:
- wire segments 252 -> 254
- no-connect marks 1 -> 0
Changed lines of the file:
@@
 Wire Wire Line
 	3200 2150 4250 2150
-NoConn ~ 5050 5500
-Text Notes 4500 5700 0    50   ~ 0
+Text Notes 4550 5850 0    50   ~ 0
 Calibration can be done via SPI
 Wire Wire Line
@@
 Connection ~ 10100 2750
 Connection ~ 10100 5600
+$Comp
+L power:GND #PWR0136
+U 1 1 5BADAC6F
+P 4950 5600
+F 0 "#PWR0136" H 4950 5350 50  0001 C CNN
+F 1 "GND" H 4950 5450 50  0000 C CNN
+F 2 "" H 4950 5600 50  0001 C CNN
+F 3 "" H 4950 5600 50  0001 C CNN
+	1    4950 5600
+	1    0    0    -1
+$EndComp
+Wire Wire Line
+	4950 5600 4950 5500
+Wire Wire Line
+	4950 5500 5050 5500
 $EndSCHEMATC
