File: kicad/micro-motor-v2/Microcontroller.sch (KiCad schematic (older format))
At the start: 10 parts

Commit message: micro-motor-v2: Schematic continued
Parts:
- added C? (x5): 100n, symbol Device:C
- added D?: POWER/blue, symbol Device:LED
- added D?: DAC1/red, symbol Device:LED
- added D?: DAC2/green, symbol Device:LED
- added J?: USB_B_Micro, symbol Connector:USB_B_Micro
- added J?: UART, symbol Connector_Generic_MountingPin:Conn_01x03_MountingPin
- added J?: SWD, symbol Connector_Generic_MountingPin:Conn_01x03_MountingPin
- added R?: 20k, symbol Device:R
- added R? (x4): 1k, symbol Device:R
- added TP?: BK, symbol Connector:TestPoint
- added TP?: DAC1, symbol Connector:TestPoint
- added TP?: DAC2, symbol Connector:TestPoint
- TH?: value Thermistor_NTC -> NTC
Connections:
- net +3V3: now also U?.1 (VBAT), U?.21 (VDDA), U?.24 (VDD), U?.36 (VDD), U?.48 (VDD), C?.1, C?.1, C?.1, R?.1
- net GND: now also U?.19 (VSSA), U?.23 (VSS), U?.35 (VSS), U?.47 (VSS), C?.2, C?.2, C?.2, C?.2, C?.2, D?.1 (K), D?.1 (K), D?.1 (K), J?.1 (Pin_1), J?.2 (Pin_2), J?.5 (GND), J?.6 (Shield), J?.MP (MountPin), J?.MP (MountPin), R?.2
- net HALL_U: now also U?.2 (PC13/RTC_OUT1/RTC_TAMP1/RTC_TS/SYS_WKUP2/TIM1_BKIN/TIM1_CH1N/TIM8_CH4N); no longer U?.37 (PA13/I2C1_SCL/I2C4_SCL/IR_OUT/SAI1_SD_B/SYS_JTMS-SWDIO/TIM16_CH1N/TIM4_CH3/USART3_CTS/USART3_NSS)
- net HALL_V: now also U?.3 (PC14-OSC32_IN/RCC_OSC32_IN); no longer U?.38 (PA14/I2C1_SDA/I2C4_SMBA/LPTIM1_OUT/SAI1_FS_B/SYS_JTCK-SWCLK/TIM1_BKIN/TIM8_CH2/USART2_TX)
- net HALL_W: now also U?.4 (PC15-OSC32_OUT/ADC1_EXTI15/ADC2_EXTI15/RCC_OSC32_OUT); no longer U?.39 (PA15/ADC1_EXTI15/ADC2_EXTI15/FDCAN3_TX/HRTIM1_FLT2/I2C1_SCL/I2S3_WS/SPI1_NSS/SPI3_NSS/SYS_JTDI/TIM1_BKIN/TIM2_CH1/TIM2_ETR/TIM8_CH1/USART2_RX)
- net BK: now reaches U?.10 (PA2/ADC1_IN3/ADC3_EXTI2/ADC4_EXTI2/ADC5_EXTI2/COMP2_INM/COMP2_OUT/LPUART1_TX/OPAMP1_VOUT/QUADSPI1_BK1_NCS/RCC_LSCO/SYS_WKUP4/TIM15_CH1/TIM2_CH3/TIM5_CH3/UCPD1_FRSTX1/UCPD1_FRSTX2/USART2_TX)
- net BK: now also TP?.1
- net Curr_W: now reaches U?.11 (PA3/ADC1_IN4/ADC3_EXTI3/ADC4_EXTI3/ADC5_EXTI3/COMP2_INP/LPUART1_RX/OPAMP1_VINM/OPAMP1_VINM0/OPAMP1_VINM1/OPAMP1_VINM_SEC/OPAMP1_VINP/OPAMP1_VINP_SEC/OPAMP5_VINM/OPAMP5_VINM0/OPAMP5_VINM1/OPAMP5_VINM_SEC/QUADSPI1_CLK/SAI1_CK1/SAI1_MCLK_A/TIM15_CH2/TIM2_CH4/TIM5_CH4/USART2_RX)
- net DAC1: now reaches U?.12 (PA4/ADC2_IN17/COMP1_INM/DAC1_OUT1/I2S3_WS/SAI1_FS_B/SPI1_NSS/SPI3_NSS/TIM3_CH2/USART2_CK)
- net DAC1: now also R?.1, TP?.1
- net DAC2: now reaches U?.13 (PA5/ADC2_IN13/COMP2_INM/DAC1_OUT2/OPAMP2_VINM/OPAMP2_VINM0/OPAMP2_VINM1/OPAMP2_VINM_SEC/SPI1_SCK/TIM2_CH1/TIM2_ETR/UCPD1_FRSTX1/UCPD1_FRSTX2)
- net DAC2: now also R?.1, TP?.1
- net Volt_U: now reaches U?.14 (PA6/ADC2_IN3/COMP1_OUT/DAC2_OUT1/LPUART1_CTS/OPAMP2_VOUT/QUADSPI1_BK1_IO3/SPI1_MISO/TIM16_CH1/TIM1_BKIN/TIM3_CH1/TIM8_BKIN)
- net Volt_V: now reaches U?.15 (PA7/ADC2_IN4/COMP2_INP/COMP2_OUT/OPAMP1_VINP/OPAMP1_VINP_SEC/OPAMP2_VINP/OPAMP2_VINP_SEC/QUADSPI1_BK1_IO2/SPI1_MOSI/TIM17_CH1/TIM1_CH1N/TIM3_CH2/TIM8_CH1N/UCPD1_FRSTX1/UCPD1_FRSTX2)
- net USB_D-: now reaches U?.33 (PA11/ADC1_EXTI11/ADC2_EXTI11/COMP1_OUT/FDCAN1_RX/HRTIM1_CHB2/I2S2_SD/SPI2_MOSI/TIM1_BKIN2/TIM1_CH1N/TIM1_CH4/TIM4_CH1/USART1_CTS/USART1_NSS/USB_DM)
- net USB_D-: now also J?.2 (D-)
- net USB_D+: now reaches U?.34 (PA12/COMP2_OUT/FDCAN1_TX/HRTIM1_FLT1/I2S_CKIN/TIM16_CH1/TIM1_CH2N/TIM1_ETR/TIM4_CH2/USART1_DE/USART1_RTS/USB_DP)
- net USB_D+: now also J?.3 (D+)
- net Curr_U: now reaches U?.8 (PA0/ADC1_IN1/ADC2_IN1/COMP1_INM/COMP1_OUT/COMP3_INP/RTC_TAMP2/SYS_WKUP1/TIM2_CH1/TIM2_ETR/TIM5_CH1/TIM8_BKIN/TIM8_ETR/USART2_CTS/USART2_NSS)
- net Curr_V: now reaches U?.9 (PA1/ADC1_IN2/ADC2_IN2/COMP1_INP/OPAMP1_VINP/OPAMP1_VINP_SEC/OPAMP3_VINP/OPAMP3_VINP_SEC/OPAMP6_VINM/OPAMP6_VINM0/OPAMP6_VINM1/OPAMP6_VINM_SEC/RTC_REFIN/TIM15_CH1N/TIM2_CH2/TIM5_CH2/USART2_DE/USART2_RTS)
- net Volt_W: now reaches U?.16 (PB0/ADC1_IN15/ADC3_IN12/COMP4_INP/HRTIM1_FLT5/OPAMP2_VINP/OPAMP2_VINP_SEC/OPAMP3_VINP/OPAMP3_VINP_SEC/QUADSPI1_BK1_IO1/TIM1_CH2N/TIM3_CH3/TIM8_CH2N/UCPD1_FRSTX1/UCPD1_FRSTX2)
- net ADC_Vsupply: now reaches U?.17 (PB1/ADC1_IN12/ADC3_IN1/COMP1_INP/COMP4_OUT/HRTIM1_SCOUT/LPUART1_DE/LPUART1_RTS/OPAMP3_VOUT/OPAMP6_VINM/OPAMP6_VINM0/OPAMP6_VINM1/OPAMP6_VINM_SEC/QUADSPI1_BK1_IO0/TIM1_CH3N/TIM3_CH4/TIM8_CH3N)
- net ADC_Vsupply: now also R?.1, R?.2
- net ADC_NTC: now reaches R?.2, TH?.1, U?.18 (PB2/ADC2_IN12/ADC3_EXTI2/ADC4_EXTI2/ADC5_EXTI2/COMP4_INM/HRTIM1_SCIN/I2C3_SMBA/LPTIM1_OUT/OPAMP3_VINM/OPAMP3_VINM0/OPAMP3_VINM1/OPAMP3_VINM_SEC/QUADSPI1_BK2_IO1/RTC_OUT2/TIM20_CH1/TIM5_CH1)
- net SPI_MOSI: now reaches U?.22 (PB10/COMP5_INM/DAC1_EXTI10/DAC2_EXTI10/DAC3_EXTI10/DAC4_EXTI10/HRTIM1_FLT3/LPUART1_RX/OPAMP3_VINM/OPAMP3_VINM0/OPAMP3_VINM1/OPAMP3_VINM_SEC/OPAMP4_VINM/OPAMP4_VINM0/OPAMP4_VINM1/OPAMP4_VINM_SEC/QUADSPI1_CLK/SAI1_SCK_A/TIM1_BKIN/TIM2_CH3/USART3_TX)
- net SPI_MISO: now reaches U?.25 (PB11/ADC1_EXTI11/ADC1_IN14/ADC2_EXTI11/ADC2_IN14/COMP6_INP/HRTIM1_FLT4/LPUART1_TX/OPAMP4_VINP/OPAMP4_VINP_SEC/OPAMP6_VOUT/QUADSPI1_BK1_NCS/TIM2_CH4/USART3_RX)
- net SPI_SCK: now reaches U?.26 (PB12/ADC1_IN11/ADC4_IN3/COMP7_INM/FDCAN2_RX/HRTIM1_CHC1/I2C2_SMBA/I2S2_WS/LPUART1_DE/LPUART1_RTS/OPAMP4_VOUT/OPAMP6_VINP/OPAMP6_VINP_SEC/SPI2_NSS/TIM1_BKIN/TIM5_ETR/USART3_CK)
- net UART_TX: now reaches U?.43 (PB6/COMP4_OUT/FDCAN2_TX/HRTIM1_EEV4/HRTIM1_SCIN/LPTIM1_ETR/SAI1_FS_B/TIM16_CH1N/TIM4_CH1/TIM8_BKIN2/TIM8_CH1/TIM8_ETR/UCPD1_CC1/USART1_TX)
- net UART_TX: now also J?.3 (Pin_3)
- net UART_RX: now reaches U?.44 (PB7/COMP3_OUT/HRTIM1_EEV3/I2C1_SDA/I2C4_SDA/LPTIM1_IN2/SYS_PVD_IN/TIM17_CH1N/TIM3_CH4/TIM4_CH2/TIM8_BKIN/USART1_RX)
- net UART_RX: now also J?.2 (Pin_2)
- net ENABLE: now reaches U?.5 (PF0-OSC_IN/ADC1_IN10/I2C2_SDA/I2S2_WS/RCC_OSC_IN/SPI2_NSS/TIM1_CH3N)
- net ~CS: now reaches U?.6 (PF1-OSC_OUT/ADC2_IN10/COMP3_INM/I2S2_CK/RCC_OSC_OUT/SPI2_SCK)
- net NRST: now reaches U?.7 (PG10-NRST/DAC1_EXTI10/DAC2_EXTI10/DAC3_EXTI10/DAC4_EXTI10/RCC_MCO)
- net NRST: now also C?.1
- net VREF: now reaches U?.20 (VREF+/VREFBUF_OUT)
- net VREF: now also C?.1
- net INDEX_I renamed INDEX
- new net: D?.2 (A), R?.2 (x3)
- new net +24V: R?.1
- new net SWCLK: J?.1 (Pin_1), U?.38 (PA14/I2C1_SDA/I2C4_SMBA/LPTIM1_OUT/SAI1_FS_B/SYS_JTCK-SWCLK/TIM1_BKIN/TIM8_CH2/USART2_TX)
- new net SWDIO: J?.3 (Pin_3), U?.37 (PA13/I2C1_SCL/I2C4_SCL/IR_OUT/SAI1_SD_B/SYS_JTMS-SWDIO/TIM16_CH1N/TIM4_CH3/USART3_CTS/USART3_NSS)
- new net SWITCH: U?.39 (PA15/ADC1_EXTI15/ADC2_EXTI15/FDCAN3_TX/HRTIM1_FLT2/I2C1_SCL/I2S3_WS/SPI1_NSS/SPI3_NSS/SYS_JTDI/TIM1_BKIN/TIM2_CH1/TIM2_ETR/TIM8_CH1/USART2_RX)
- no-connect marks 0 -> 2
Other:
- note added: "Debug LEDs"
- note added: "Decoupling capacitors for MCU"
- moved on the sheet: R?, TH?, U?B, U?C, U?D, U?E, U?F, U?G, U?H

Commit message: micro-motor-v2: Schematic finished
Parts:
- removed R?: 20k, symbol Device:R
- removed R?: 1k, symbol Device:R
- removed R?: 10k, symbol Device:R
- removed TH?: NTC, symbol Device:Thermistor_NTC
- added C306: 100n, Capacitor_SMD:C_0402_1005Metric, symbol Device:C
- C301, C302, C303, C304, C305: renamed from C?; footprint (none) -> Capacitor_SMD:C_0402_1005Metric
- D301, D302, D303: renamed from D?; footprint (none) -> LED_SMD:LED_0402_1005Metric
- J301: renamed from J?; value USB_B_Micro -> USB; footprint (none) -> Connector_USB:USB_Micro-B_Molex-105133-0001
- J302, J303: renamed from J?; footprint (none) -> Connector_JST:JST_GH_BM03B-GHS-TBT_1x03-1MP_P1.25mm_Vertical
- R304, R305, R306: renamed from R?; footprint (none) -> Resistor_SMD:R_0402_1005Metric
- TP301, TP302, TP303: renamed from TP?; footprint (none) -> TestPoint:TestPoint_Pad_D1.0mm
- U301: renamed from U?; value STM32G474C(B-C-E)Tx_u -> STM32G474CET6; footprint LQFP48 -> Package_QFP:LQFP-48_7x7mm_P0.5mm
Connections:
- net +3V3: now also U301.1 (VBAT), U301.21 (VDDA), U301.24 (VDD), U301.36 (VDD), U301.48 (VDD), C306.1; no longer U301.1 (VBAT), U301.21 (VDDA), U301.24 (VDD), U301.36 (VDD), U301.48 (VDD)
- net A: now also U301.42 (PB5/FDCAN2_RX/HRTIM1_EEV6/I2C1_SMBA/I2C3_SDA/I2S3_SD/LPTIM1_IN1/SAI1_SD_B/SPI1_MOSI/SPI3_MOSI/TIM16_BKIN/TIM17_CH1/TIM3_CH2/TIM8_CH3N/USART2_CK); no longer U301.42 (PB5/FDCAN2_RX/HRTIM1_EEV6/I2C1_SMBA/I2C3_SDA/I2S3_SD/LPTIM1_IN1/SAI1_SD_B/SPI1_MOSI/SPI3_MOSI/TIM16_BKIN/TIM17_CH1/TIM3_CH2/TIM8_CH3N/USART2_CK)
- net ADC_NTC: now also U301.18 (PB2/ADC2_IN12/ADC3_EXTI2/ADC4_EXTI2/ADC5_EXTI2/COMP4_INM/HRTIM1_SCIN/I2C3_SMBA/LPTIM1_OUT/OPAMP3_VINM/OPAMP3_VINM0/OPAMP3_VINM1/OPAMP3_VINM_SEC/QUADSPI1_BK2_IO1/RTC_OUT2/TIM20_CH1/TIM5_CH1); no longer U301.18 (PB2/ADC2_IN12/ADC3_EXTI2/ADC4_EXTI2/ADC5_EXTI2/COMP4_INM/HRTIM1_SCIN/I2C3_SMBA/LPTIM1_OUT/OPAMP3_VINM/OPAMP3_VINM0/OPAMP3_VINM1/OPAMP3_VINM_SEC/QUADSPI1_BK2_IO1/RTC_OUT2/TIM20_CH1/TIM5_CH1)
- net ADC_Vsupply: now also U301.17 (PB1/ADC1_IN12/ADC3_IN1/COMP1_INP/COMP4_OUT/HRTIM1_SCOUT/LPUART1_DE/LPUART1_RTS/OPAMP3_VOUT/OPAMP6_VINM/OPAMP6_VINM0/OPAMP6_VINM1/OPAMP6_VINM_SEC/QUADSPI1_BK1_IO0/TIM1_CH3N/TIM3_CH4/TIM8_CH3N); no longer U301.17 (PB1/ADC1_IN12/ADC3_IN1/COMP1_INP/COMP4_OUT/HRTIM1_SCOUT/LPUART1_DE/LPUART1_RTS/OPAMP3_VOUT/OPAMP6_VINM/OPAMP6_VINM0/OPAMP6_VINM1/OPAMP6_VINM_SEC/QUADSPI1_BK1_IO0/TIM1_CH3N/TIM3_CH4/TIM8_CH3N)
- net B: now also U301.41 (PB4/FDCAN3_TX/HRTIM1_EEV7/SAI1_MCLK_B/SPI1_MISO/SPI3_MISO/SYS_JTRST/TIM16_CH1/TIM17_BKIN/TIM3_CH1/TIM8_CH2N/UCPD1_CC2/USART2_RX); no longer U301.41 (PB4/FDCAN3_TX/HRTIM1_EEV7/SAI1_MCLK_B/SPI1_MISO/SPI3_MISO/SYS_JTRST/TIM16_CH1/TIM17_BKIN/TIM3_CH1/TIM8_CH2N/UCPD1_CC2/USART2_RX)
- net BK: now also U301.10 (PA2/ADC1_IN3/ADC3_EXTI2/ADC4_EXTI2/ADC5_EXTI2/COMP2_INM/COMP2_OUT/LPUART1_TX/OPAMP1_VOUT/QUADSPI1_BK1_NCS/RCC_LSCO/SYS_WKUP4/TIM15_CH1/TIM2_CH3/TIM5_CH3/UCPD1_FRSTX1/UCPD1_FRSTX2/USART2_TX); no longer U301.10 (PA2/ADC1_IN3/ADC3_EXTI2/ADC4_EXTI2/ADC5_EXTI2/COMP2_INM/COMP2_OUT/LPUART1_TX/OPAMP1_VOUT/QUADSPI1_BK1_NCS/RCC_LSCO/SYS_WKUP4/TIM15_CH1/TIM2_CH3/TIM5_CH3/UCPD1_FRSTX1/UCPD1_FRSTX2/USART2_TX)
- net CAN_RX: now also U301.45 (PB8-BOOT0/COMP1_OUT/FDCAN1_RX/HRTIM1_EEV8/I2C1_SCL/SAI1_CK1/SAI1_MCLK_A/TIM16_CH1/TIM1_BKIN/TIM4_CH3/TIM8_CH2/USART3_RX); no longer U301.45 (PB8-BOOT0/COMP1_OUT/FDCAN1_RX/HRTIM1_EEV8/I2C1_SCL/SAI1_CK1/SAI1_MCLK_A/TIM16_CH1/TIM1_BKIN/TIM4_CH3/TIM8_CH2/USART3_RX)
- net CAN_TX: now also U301.46 (PB9/COMP2_OUT/DAC1_EXTI9/DAC2_EXTI9/DAC3_EXTI9/DAC4_EXTI9/FDCAN1_TX/HRTIM1_EEV5/I2C1_SDA/IR_OUT/SAI1_D2/SAI1_FS_A/TIM17_CH1/TIM1_CH3N/TIM4_CH4/TIM8_CH3/USART3_TX); no longer U301.46 (PB9/COMP2_OUT/DAC1_EXTI9/DAC2_EXTI9/DAC3_EXTI9/DAC4_EXTI9/FDCAN1_TX/HRTIM1_EEV5/I2C1_SDA/IR_OUT/SAI1_D2/SAI1_FS_A/TIM17_CH1/TIM1_CH3N/TIM4_CH4/TIM8_CH3/USART3_TX)
- net Curr_U: now also U301.8 (PA0/ADC1_IN1/ADC2_IN1/COMP1_INM/COMP1_OUT/COMP3_INP/RTC_TAMP2/SYS_WKUP1/TIM2_CH1/TIM2_ETR/TIM5_CH1/TIM8_BKIN/TIM8_ETR/USART2_CTS/USART2_NSS); no longer U301.8 (PA0/ADC1_IN1/ADC2_IN1/COMP1_INM/COMP1_OUT/COMP3_INP/RTC_TAMP2/SYS_WKUP1/TIM2_CH1/TIM2_ETR/TIM5_CH1/TIM8_BKIN/TIM8_ETR/USART2_CTS/USART2_NSS)
- net Curr_V: now also U301.9 (PA1/ADC1_IN2/ADC2_IN2/COMP1_INP/OPAMP1_VINP/OPAMP1_VINP_SEC/OPAMP3_VINP/OPAMP3_VINP_SEC/OPAMP6_VINM/OPAMP6_VINM0/OPAMP6_VINM1/OPAMP6_VINM_SEC/RTC_REFIN/TIM15_CH1N/TIM2_CH2/TIM5_CH2/USART2_DE/USART2_RTS); no longer U301.9 (PA1/ADC1_IN2/ADC2_IN2/COMP1_INP/OPAMP1_VINP/OPAMP1_VINP_SEC/OPAMP3_VINP/OPAMP3_VINP_SEC/OPAMP6_VINM/OPAMP6_VINM0/OPAMP6_VINM1/OPAMP6_VINM_SEC/RTC_REFIN/TIM15_CH1N/TIM2_CH2/TIM5_CH2/USART2_DE/USART2_RTS)
- net Curr_W: now also U301.11 (PA3/ADC1_IN4/ADC3_EXTI3/ADC4_EXTI3/ADC5_EXTI3/COMP2_INP/LPUART1_RX/OPAMP1_VINM/OPAMP1_VINM0/OPAMP1_VINM1/OPAMP1_VINM_SEC/OPAMP1_VINP/OPAMP1_VINP_SEC/OPAMP5_VINM/OPAMP5_VINM0/OPAMP5_VINM1/OPAMP5_VINM_SEC/QUADSPI1_CLK/SAI1_CK1/SAI1_MCLK_A/TIM15_CH2/TIM2_CH4/TIM5_CH4/USART2_RX); no longer U301.11 (PA3/ADC1_IN4/ADC3_EXTI3/ADC4_EXTI3/ADC5_EXTI3/COMP2_INP/LPUART1_RX/OPAMP1_VINM/OPAMP1_VINM0/OPAMP1_VINM1/OPAMP1_VINM_SEC/OPAMP1_VINP/OPAMP1_VINP_SEC/OPAMP5_VINM/OPAMP5_VINM0/OPAMP5_VINM1/OPAMP5_VINM_SEC/QUADSPI1_CLK/SAI1_CK1/SAI1_MCLK_A/TIM15_CH2/TIM2_CH4/TIM5_CH4/USART2_RX)
- net DAC1: now also U301.12 (PA4/ADC2_IN17/COMP1_INM/DAC1_OUT1/I2S3_WS/SAI1_FS_B/SPI1_NSS/SPI3_NSS/TIM3_CH2/USART2_CK); no longer U301.12 (PA4/ADC2_IN17/COMP1_INM/DAC1_OUT1/I2S3_WS/SAI1_FS_B/SPI1_NSS/SPI3_NSS/TIM3_CH2/USART2_CK)
- net DAC2: now also U301.13 (PA5/ADC2_IN13/COMP2_INM/DAC1_OUT2/OPAMP2_VINM/OPAMP2_VINM0/OPAMP2_VINM1/OPAMP2_VINM_SEC/SPI1_SCK/TIM2_CH1/TIM2_ETR/UCPD1_FRSTX1/UCPD1_FRSTX2); no longer U301.13 (PA5/ADC2_IN13/COMP2_INM/DAC1_OUT2/OPAMP2_VINM/OPAMP2_VINM0/OPAMP2_VINM1/OPAMP2_VINM_SEC/SPI1_SCK/TIM2_CH1/TIM2_ETR/UCPD1_FRSTX1/UCPD1_FRSTX2)
- net ENABLE: now also U301.5 (PF0-OSC_IN/ADC1_IN10/I2C2_SDA/I2S2_WS/RCC_OSC_IN/SPI2_NSS/TIM1_CH3N); no longer U301.5 (PF0-OSC_IN/ADC1_IN10/I2C2_SDA/I2S2_WS/RCC_OSC_IN/SPI2_NSS/TIM1_CH3N)
- net GND: now also C306.2
- net INDEX: now also U301.40 (PB3/ADC3_EXTI3/ADC4_EXTI3/ADC5_EXTI3/CRS_SYNC/FDCAN3_RX/HRTIM1_EEV9/HRTIM1_SCOUT/I2S3_CK/SAI1_SCK_B/SPI1_SCK/SPI3_SCK/SYS_JTDO-SWO/TIM2_CH2/TIM3_ETR/TIM4_ETR/TIM8_CH1N/USART2_TX); no longer U301.40 (PB3/ADC3_EXTI3/ADC4_EXTI3/ADC5_EXTI3/CRS_SYNC/FDCAN3_RX/HRTIM1_EEV9/HRTIM1_SCOUT/I2S3_CK/SAI1_SCK_B/SPI1_SCK/SPI3_SCK/SYS_JTDO-SWO/TIM2_CH2/TIM3_ETR/TIM4_ETR/TIM8_CH1N/USART2_TX)
- net NRST: now also U301.7 (PG10-NRST/DAC1_EXTI10/DAC2_EXTI10/DAC3_EXTI10/DAC4_EXTI10/RCC_MCO); no longer U301.7 (PG10-NRST/DAC1_EXTI10/DAC2_EXTI10/DAC3_EXTI10/DAC4_EXTI10/RCC_MCO)
- net PWM_CH1N: now also U301.27 (PB13/ADC3_IN5/COMP5_INP/FDCAN2_TX/HRTIM1_CHC2/I2S2_CK/LPUART1_CTS/OPAMP3_VINP/OPAMP3_VINP_SEC/OPAMP4_VINP/OPAMP4_VINP_SEC/OPAMP6_VINP/OPAMP6_VINP_SEC/SPI2_SCK/TIM1_CH1N/USART3_CTS/USART3_NSS); no longer U301.27 (PB13/ADC3_IN5/COMP5_INP/FDCAN2_TX/HRTIM1_CHC2/I2S2_CK/LPUART1_CTS/OPAMP3_VINP/OPAMP3_VINP_SEC/OPAMP4_VINP/OPAMP4_VINP_SEC/OPAMP6_VINP/OPAMP6_VINP_SEC/SPI2_SCK/TIM1_CH1N/USART3_CTS/USART3_NSS)
- net PWM_CH1P: now also U301.30 (PA8/ADC5_IN1/COMP7_OUT/FDCAN3_RX/HRTIM1_CHA1/I2C2_SDA/I2C3_SCL/I2S2_MCK/OPAMP5_VOUT/RCC_MCO/SAI1_CK2/SAI1_SCK_A/TIM1_CH1/TIM4_ETR/USART1_CK); no longer U301.30 (PA8/ADC5_IN1/COMP7_OUT/FDCAN3_RX/HRTIM1_CHA1/I2C2_SDA/I2C3_SCL/I2S2_MCK/OPAMP5_VOUT/RCC_MCO/SAI1_CK2/SAI1_SCK_A/TIM1_CH1/TIM4_ETR/USART1_CK)
- net PWM_CH2N: now also U301.28 (PB14/ADC1_IN5/ADC4_IN4/COMP4_OUT/COMP7_INP/HRTIM1_CHD1/OPAMP2_VINP/OPAMP2_VINP_SEC/OPAMP5_VINP/OPAMP5_VINP_SEC/SPI2_MISO/TIM15_CH1/TIM1_CH2N/USART3_DE/USART3_RTS); no longer U301.28 (PB14/ADC1_IN5/ADC4_IN4/COMP4_OUT/COMP7_INP/HRTIM1_CHD1/OPAMP2_VINP/OPAMP2_VINP_SEC/OPAMP5_VINP/OPAMP5_VINP_SEC/SPI2_MISO/TIM15_CH1/TIM1_CH2N/USART3_DE/USART3_RTS)
- net PWM_CH2P: now also U301.31 (PA9/ADC5_IN2/COMP5_OUT/DAC1_EXTI9/DAC2_EXTI9/DAC3_EXTI9/DAC4_EXTI9/HRTIM1_CHA2/I2C2_SCL/I2C3_SMBA/I2S3_MCK/SAI1_FS_A/TIM15_BKIN/TIM1_CH2/TIM2_CH3/UCPD1_DBCC1/USART1_TX); no longer U301.31 (PA9/ADC5_IN2/COMP5_OUT/DAC1_EXTI9/DAC2_EXTI9/DAC3_EXTI9/DAC4_EXTI9/HRTIM1_CHA2/I2C2_SCL/I2C3_SMBA/I2S3_MCK/SAI1_FS_A/TIM15_BKIN/TIM1_CH2/TIM2_CH3/UCPD1_DBCC1/USART1_TX)
- net PWM_CH3N: now also U301.29 (PB15/ADC1_EXTI15/ADC2_EXTI15/ADC2_IN15/ADC4_IN5/COMP3_OUT/COMP6_INM/HRTIM1_CHD2/I2S2_SD/OPAMP5_VINM/OPAMP5_VINM0/OPAMP5_VINM1/OPAMP5_VINM_SEC/RTC_REFIN/SPI2_MOSI/TIM15_CH1N/TIM15_CH2/TIM1_CH3N); no longer U301.29 (PB15/ADC1_EXTI15/ADC2_EXTI15/ADC2_IN15/ADC4_IN5/COMP3_OUT/COMP6_INM/HRTIM1_CHD2/I2S2_SD/OPAMP5_VINM/OPAMP5_VINM0/OPAMP5_VINM1/OPAMP5_VINM_SEC/RTC_REFIN/SPI2_MOSI/TIM15_CH1N/TIM15_CH2/TIM1_CH3N)
- net PWM_CH3P: now also U301.32 (PA10/COMP6_OUT/CRS_SYNC/DAC1_EXTI10/DAC2_EXTI10/DAC3_EXTI10/DAC4_EXTI10/HRTIM1_CHB1/I2C2_SMBA/SAI1_D1/SAI1_SD_A/SPI2_MISO/TIM17_BKIN/TIM1_CH3/TIM2_CH4/TIM8_BKIN/UCPD1_DBCC2/USART1_RX); no longer U301.32 (PA10/COMP6_OUT/CRS_SYNC/DAC1_EXTI10/DAC2_EXTI10/DAC3_EXTI10/DAC4_EXTI10/HRTIM1_CHB1/I2C2_SMBA/SAI1_D1/SAI1_SD_A/SPI2_MISO/TIM17_BKIN/TIM1_CH3/TIM2_CH4/TIM8_BKIN/UCPD1_DBCC2/USART1_RX)
- net SPI_MISO: now also U301.25 (PB11/ADC1_EXTI11/ADC1_IN14/ADC2_EXTI11/ADC2_IN14/COMP6_INP/HRTIM1_FLT4/LPUART1_TX/OPAMP4_VINP/OPAMP4_VINP_SEC/OPAMP6_VOUT/QUADSPI1_BK1_NCS/TIM2_CH4/USART3_RX); no longer U301.25 (PB11/ADC1_EXTI11/ADC1_IN14/ADC2_EXTI11/ADC2_IN14/COMP6_INP/HRTIM1_FLT4/LPUART1_TX/OPAMP4_VINP/OPAMP4_VINP_SEC/OPAMP6_VOUT/QUADSPI1_BK1_NCS/TIM2_CH4/USART3_RX)
- net SPI_MOSI: now also U301.22 (PB10/COMP5_INM/DAC1_EXTI10/DAC2_EXTI10/DAC3_EXTI10/DAC4_EXTI10/HRTIM1_FLT3/LPUART1_RX/OPAMP3_VINM/OPAMP3_VINM0/OPAMP3_VINM1/OPAMP3_VINM_SEC/OPAMP4_VINM/OPAMP4_VINM0/OPAMP4_VINM1/OPAMP4_VINM_SEC/QUADSPI1_CLK/SAI1_SCK_A/TIM1_BKIN/TIM2_CH3/USART3_TX); no longer U301.22 (PB10/COMP5_INM/DAC1_EXTI10/DAC2_EXTI10/DAC3_EXTI10/DAC4_EXTI10/HRTIM1_FLT3/LPUART1_RX/OPAMP3_VINM/OPAMP3_VINM0/OPAMP3_VINM1/OPAMP3_VINM_SEC/OPAMP4_VINM/OPAMP4_VINM0/OPAMP4_VINM1/OPAMP4_VINM_SEC/QUADSPI1_CLK/SAI1_SCK_A/TIM1_BKIN/TIM2_CH3/USART3_TX)
- net SPI_SCK: now also U301.26 (PB12/ADC1_IN11/ADC4_IN3/COMP7_INM/FDCAN2_RX/HRTIM1_CHC1/I2C2_SMBA/I2S2_WS/LPUART1_DE/LPUART1_RTS/OPAMP4_VOUT/OPAMP6_VINP/OPAMP6_VINP_SEC/SPI2_NSS/TIM1_BKIN/TIM5_ETR/USART3_CK); no longer U301.26 (PB12/ADC1_IN11/ADC4_IN3/COMP7_INM/FDCAN2_RX/HRTIM1_CHC1/I2C2_SMBA/I2S2_WS/LPUART1_DE/LPUART1_RTS/OPAMP4_VOUT/OPAMP6_VINP/OPAMP6_VINP_SEC/SPI2_NSS/TIM1_BKIN/TIM5_ETR/USART3_CK)
- net SWCLK: now also U301.38 (PA14/I2C1_SDA/I2C4_SMBA/LPTIM1_OUT/SAI1_FS_B/SYS_JTCK-SWCLK/TIM1_BKIN/TIM8_CH2/USART2_TX); no longer U301.38 (PA14/I2C1_SDA/I2C4_SMBA/LPTIM1_OUT/SAI1_FS_B/SYS_JTCK-SWCLK/TIM1_BKIN/TIM8_CH2/USART2_TX)
- net SWDIO: now also U301.37 (PA13/I2C1_SCL/I2C4_SCL/IR_OUT/SAI1_SD_B/SYS_JTMS-SWDIO/TIM16_CH1N/TIM4_CH3/USART3_CTS/USART3_NSS); no longer U301.37 (PA13/I2C1_SCL/I2C4_SCL/IR_OUT/SAI1_SD_B/SYS_JTMS-SWDIO/TIM16_CH1N/TIM4_CH3/USART3_CTS/USART3_NSS)
- net SWITCH: now also U301.39 (PA15/ADC1_EXTI15/ADC2_EXTI15/FDCAN3_TX/HRTIM1_FLT2/I2C1_SCL/I2S3_WS/SPI1_NSS/SPI3_NSS/SYS_JTDI/TIM1_BKIN/TIM2_CH1/TIM2_ETR/TIM8_CH1/USART2_RX); no longer U301.39 (PA15/ADC1_EXTI15/ADC2_EXTI15/FDCAN3_TX/HRTIM1_FLT2/I2C1_SCL/I2S3_WS/SPI1_NSS/SPI3_NSS/SYS_JTDI/TIM1_BKIN/TIM2_CH1/TIM2_ETR/TIM8_CH1/USART2_RX)
- net UART_RX: now also U301.44 (PB7/COMP3_OUT/HRTIM1_EEV3/I2C1_SDA/I2C4_SDA/LPTIM1_IN2/SYS_PVD_IN/TIM17_CH1N/TIM3_CH4/TIM4_CH2/TIM8_BKIN/USART1_RX); no longer U301.44 (PB7/COMP3_OUT/HRTIM1_EEV3/I2C1_SDA/I2C4_SDA/LPTIM1_IN2/SYS_PVD_IN/TIM17_CH1N/TIM3_CH4/TIM4_CH2/TIM8_BKIN/USART1_RX)
- net UART_TX: now also U301.43 (PB6/COMP4_OUT/FDCAN2_TX/HRTIM1_EEV4/HRTIM1_SCIN/LPTIM1_ETR/SAI1_FS_B/TIM16_CH1N/TIM4_CH1/TIM8_BKIN2/TIM8_CH1/TIM8_ETR/UCPD1_CC1/USART1_TX); no longer U301.43 (PB6/COMP4_OUT/FDCAN2_TX/HRTIM1_EEV4/HRTIM1_SCIN/LPTIM1_ETR/SAI1_FS_B/TIM16_CH1N/TIM4_CH1/TIM8_BKIN2/TIM8_CH1/TIM8_ETR/UCPD1_CC1/USART1_TX)
- net USB_D+: now also U301.34 (PA12/COMP2_OUT/FDCAN1_TX/HRTIM1_FLT1/I2S_CKIN/TIM16_CH1/TIM1_CH2N/TIM1_ETR/TIM4_CH2/USART1_DE/USART1_RTS/USB_DP); no longer U301.34 (PA12/COMP2_OUT/FDCAN1_TX/HRTIM1_FLT1/I2S_CKIN/TIM16_CH1/TIM1_CH2N/TIM1_ETR/TIM4_CH2/USART1_DE/USART1_RTS/USB_DP)
- net USB_D-: now also U301.33 (PA11/ADC1_EXTI11/ADC2_EXTI11/COMP1_OUT/FDCAN1_RX/HRTIM1_CHB2/I2S2_SD/SPI2_MOSI/TIM1_BKIN2/TIM1_CH1N/TIM1_CH4/TIM4_CH1/USART1_CTS/USART1_NSS/USB_DM); no longer U301.33 (PA11/ADC1_EXTI11/ADC2_EXTI11/COMP1_OUT/FDCAN1_RX/HRTIM1_CHB2/I2S2_SD/SPI2_MOSI/TIM1_BKIN2/TIM1_CH1N/TIM1_CH4/TIM4_CH1/USART1_CTS/USART1_NSS/USB_DM)
- net VREF: now also U301.20 (VREF+/VREFBUF_OUT); no longer U301.20 (VREF+/VREFBUF_OUT)
- net Volt_U: now also U301.14 (PA6/ADC2_IN3/COMP1_OUT/DAC2_OUT1/LPUART1_CTS/OPAMP2_VOUT/QUADSPI1_BK1_IO3/SPI1_MISO/TIM16_CH1/TIM1_BKIN/TIM3_CH1/TIM8_BKIN); no longer U301.14 (PA6/ADC2_IN3/COMP1_OUT/DAC2_OUT1/LPUART1_CTS/OPAMP2_VOUT/QUADSPI1_BK1_IO3/SPI1_MISO/TIM16_CH1/TIM1_BKIN/TIM3_CH1/TIM8_BKIN)
- net Volt_V: now also U301.15 (PA7/ADC2_IN4/COMP2_INP/COMP2_OUT/OPAMP1_VINP/OPAMP1_VINP_SEC/OPAMP2_VINP/OPAMP2_VINP_SEC/QUADSPI1_BK1_IO2/SPI1_MOSI/TIM17_CH1/TIM1_CH1N/TIM3_CH2/TIM8_CH1N/UCPD1_FRSTX1/UCPD1_FRSTX2); no longer U301.15 (PA7/ADC2_IN4/COMP2_INP/COMP2_OUT/OPAMP1_VINP/OPAMP1_VINP_SEC/OPAMP2_VINP/OPAMP2_VINP_SEC/QUADSPI1_BK1_IO2/SPI1_MOSI/TIM17_CH1/TIM1_CH1N/TIM3_CH2/TIM8_CH1N/UCPD1_FRSTX1/UCPD1_FRSTX2)
- net Volt_W: now also U301.16 (PB0/ADC1_IN15/ADC3_IN12/COMP4_INP/HRTIM1_FLT5/OPAMP2_VINP/OPAMP2_VINP_SEC/OPAMP3_VINP/OPAMP3_VINP_SEC/QUADSPI1_BK1_IO1/TIM1_CH2N/TIM3_CH3/TIM8_CH2N/UCPD1_FRSTX1/UCPD1_FRSTX2); no longer U301.16 (PB0/ADC1_IN15/ADC3_IN12/COMP4_INP/HRTIM1_FLT5/OPAMP2_VINP/OPAMP2_VINP_SEC/OPAMP3_VINP/OPAMP3_VINP_SEC/QUADSPI1_BK1_IO1/TIM1_CH2N/TIM3_CH3/TIM8_CH2N/UCPD1_FRSTX1/UCPD1_FRSTX2)
- net ~CS: now also U301.6 (PF1-OSC_OUT/ADC2_IN10/COMP3_INM/I2S2_CK/RCC_OSC_OUT/SPI2_SCK); no longer U301.6 (PF1-OSC_OUT/ADC2_IN10/COMP3_INM/I2S2_CK/RCC_OSC_OUT/SPI2_SCK)
Other:
- moved on the sheet: J302

Commit message: micro-motor-v2: Layout...
Connections:
- net ADC_NTC: now also U301.17 (PB1/ADC1_IN12/ADC3_IN1/COMP1_INP/COMP4_OUT/HRTIM1_SCOUT/LPUART1_DE/LPUART1_RTS/OPAMP3_VOUT/OPAMP6_VINM/OPAMP6_VINM0/OPAMP6_VINM1/OPAMP6_VINM_SEC/QUADSPI1_BK1_IO0/TIM1_CH3N/TIM3_CH4/TIM8_CH3N); no longer U301.18 (PB2/ADC2_IN12/ADC3_EXTI2/ADC4_EXTI2/ADC5_EXTI2/COMP4_INM/HRTIM1_SCIN/I2C3_SMBA/LPTIM1_OUT/OPAMP3_VINM/OPAMP3_VINM0/OPAMP3_VINM1/OPAMP3_VINM_SEC/QUADSPI1_BK2_IO1/RTC_OUT2/TIM20_CH1/TIM5_CH1)
- net ADC_Vsupply: now also U301.18 (PB2/ADC2_IN12/ADC3_EXTI2/ADC4_EXTI2/ADC5_EXTI2/COMP4_INM/HRTIM1_SCIN/I2C3_SMBA/LPTIM1_OUT/OPAMP3_VINM/OPAMP3_VINM0/OPAMP3_VINM1/OPAMP3_VINM_SEC/QUADSPI1_BK2_IO1/RTC_OUT2/TIM20_CH1/TIM5_CH1); no longer U301.17 (PB1/ADC1_IN12/ADC3_IN1/COMP1_INP/COMP4_OUT/HRTIM1_SCOUT/LPUART1_DE/LPUART1_RTS/OPAMP3_VOUT/OPAMP6_VINM/OPAMP6_VINM0/OPAMP6_VINM1/OPAMP6_VINM_SEC/QUADSPI1_BK1_IO0/TIM1_CH3N/TIM3_CH4/TIM8_CH3N)
Changed lines of the file:
@@
 Text Notes 9150 8600 0    50   ~ 0
 Debug LEDs
+Text HLabel 2650 5700 0    50   Input ~ 0
+ADC_NTC
 Text HLabel 2650 5600 0    50   Input ~ 0
-ADC_NTC
-Text HLabel 2650 5700 0    50   Input ~ 0
 ADC_Vsupply
 Wire Wire Line

Commit message: micro-motor-v2: Layout...
Connections:
- net Volt_U: now also U301.16 (PB0/ADC1_IN15/ADC3_IN12/COMP4_INP/HRTIM1_FLT5/OPAMP2_VINP/OPAMP2_VINP_SEC/OPAMP3_VINP/OPAMP3_VINP_SEC/QUADSPI1_BK1_IO1/TIM1_CH2N/TIM3_CH3/TIM8_CH2N/UCPD1_FRSTX1/UCPD1_FRSTX2); no longer U301.14 (PA6/ADC2_IN3/COMP1_OUT/DAC2_OUT1/LPUART1_CTS/OPAMP2_VOUT/QUADSPI1_BK1_IO3/SPI1_MISO/TIM16_CH1/TIM1_BKIN/TIM3_CH1/TIM8_BKIN)
- net Volt_W: now also U301.14 (PA6/ADC2_IN3/COMP1_OUT/DAC2_OUT1/LPUART1_CTS/OPAMP2_VOUT/QUADSPI1_BK1_IO3/SPI1_MISO/TIM16_CH1/TIM1_BKIN/TIM3_CH1/TIM8_BKIN); no longer U301.16 (PB0/ADC1_IN15/ADC3_IN12/COMP4_INP/HRTIM1_FLT5/OPAMP2_VINP/OPAMP2_VINP_SEC/OPAMP3_VINP/OPAMP3_VINP_SEC/QUADSPI1_BK1_IO1/TIM1_CH2N/TIM3_CH3/TIM8_CH2N/UCPD1_FRSTX1/UCPD1_FRSTX2)
Changed lines of the file:
@@
 Wire Wire Line
 	3000 3100 2650 3100
-Text HLabel 2650 2500 0    50   Input ~ 0
-Volt_U
 Text HLabel 2650 2400 0    50   Input ~ 0
 Volt_V
-Text HLabel 2650 5800 0    50   Input ~ 0
+Text HLabel 2650 2500 0    50   Input ~ 0
 Volt_W
 Wire Wire Line
@@
 	14650 9400 14050 9400
 Connection ~ 14050 9400
+Text HLabel 2650 5800 0    50   Input ~ 0
+Volt_U
 $EndSCHEMATC
