File: kicad/micro-motor-v2/micro-motor-v2.sch (KiCad schematic (older format))
At the start: 23 parts, among them J101 SUPPLY, J102 SW, J103 Hall, J104 Encoder, J105 NTC, J106 Motor

Commit message: micro-motor-v2: Layout...
Connections:
- net Microcontroller/Volt_U: now also R102.2, R103.1; no longer R106.2, R107.1
- net Microcontroller/Volt_W: now also R106.2, R107.1; no longer R102.2, R103.1
- net Motordriver/OUT_U: now also R102.1; no longer R106.1
- net Motordriver/OUT_W: now also R106.1; no longer R102.1
Other:
- moved on the sheet: R102, R103, R106, R107
Changed lines of the file:
@@
 L Device:R R102
 U 1 1 5DAB2BB4
-P 9450 4650
-F 0 "R102" H 9520 4696 50  0000 L CNN
-F 1 "20k" H 9520 4605 50  0000 L CNN
-F 2 "Resistor_SMD:R_0402_1005Metric" V 9380 4650 50  0001 C CNN
-F 3 "~" H 9450 4650 50  0001 C CNN
-	1    9450 4650
+P 10350 4650
+F 0 "R102" H 10420 4696 50  0000 L CNN
+F 1 "20k" H 10420 4605 50  0000 L CNN
+F 2 "Resistor_SMD:R_0402_1005Metric" V 10280 4650 50  0001 C CNN
+F 3 "~" H 10350 4650 50  0001 C CNN
+	1    10350 4650
 	1    0    0    -1
 $EndComp
@@
 L Device:R R103
 U 1 1 5DAB2FEF
-P 9450 5350
-F 0 "R103" H 9520 5396 50  0000 L CNN
-F 1 "1k" H 9520 5305 50  0000 L CNN
-F 2 "Resistor_SMD:R_0402_1005Metric" V 9380 5350 50  0001 C CNN
-F 3 "~" H 9450 5350 50  0001 C CNN
-	1    9450 5350
+P 10350 5350
+F 0 "R103" H 10420 5396 50  0000 L CNN
+F 1 "1k" H 10420 5305 50  0000 L CNN
+F 2 "Resistor_SMD:R_0402_1005Metric" V 10280 5350 50  0001 C CNN
+F 3 "~" H 10350 5350 50  0001 C CNN
+	1    10350 5350
 	1    0    0    -1
 $EndComp
@@
 L Device:R R106
 U 1 1 5DAB42D7
-P 10350 4650
-F 0 "R106" H 10420 4696 50  0000 L CNN
-F 1 "20k" H 10420 4605 50  0000 L CNN
-F 2 "Resistor_SMD:R_0402_1005Metric" V 10280 4650 50  0001 C CNN
-F 3 "~" H 10350 4650 50  0001 C CNN
-	1    10350 4650
+P 9450 4650
+F 0 "R106" H 9520 4696 50  0000 L CNN
+F 1 "20k" H 9520 4605 50  0000 L CNN
+F 2 "Resistor_SMD:R_0402_1005Metric" V 9380 4650 50  0001 C CNN
+F 3 "~" H 9450 4650 50  0001 C CNN
+	1    9450 4650
 	1    0    0    -1
 $EndComp
@@
 L Device:R R107
 U 1 1 5DAB4DEA
-P 10350 5350
-F 0 "R107" H 10420 5396 50  0000 L CNN
-F 1 "1k" H 10420 5305 50  0000 L CNN
-F 2 "Resistor_SMD:R_0402_1005Metric" V 10280 5350 50  0001 C CNN
-F 3 "~" H 10350 5350 50  0001 C CNN
-	1    10350 5350
+P 9450 5350
+F 0 "R107" H 9520 5396 50  0000 L CNN
+F 1 "1k" H 9520 5305 50  0000 L CNN
+F 2 "Resistor_SMD:R_0402_1005Metric" V 9380 5350 50  0001 C CNN
+F 3 "~" H 9450 5350 50  0001 C CNN
+	1    9450 5350
 	1    0    0    -1
 $EndComp
