File: kicad/micro-motor-v2/Motordriver.sch (KiCad schematic (older format))
At the start: 17 parts, among them Q301 FDMD82xx, Q302 FDMD82xx, Q303 FDMD82xx

Commit message: micro-motor-v2: Schematic continued
Parts:
- removed R301, R303: 5m, Resistors_SMD:R_0805, symbol Device:R
- removed U? (x2): INA240A2PW, Package_SO:TSSOP-8_4.4x3mm_P0.65mm, symbol Amplifier_Current:INA240A2PW
- added R? (x2): 5m, Resistors_SMD:R_0805, symbol Device:R
- added TP?: Fault, symbol Connector:TestPoint
- added U? (x2): INA240A2PW, Package_SO:TSSOP-8_4.4x3mm_P0.65mm, symbol Amplifier_Current:INA240A2PW
- R?: value R -> 10k
- renumbered C304 to C?, C305 to C?, C302 to C?, C301 to C?, C303 to C?, C306 to C?, Q303 to Q?, Q301 to Q?, Q302 to Q?, R302 to R?
Connections:
- net +3V3: now also U?.5 (V+), U?.5 (V+), U?.5 (V+)
- net GND: now also U?.3 (-), R?.2, R?.2, U?.1 (GND), U?.1 (GND), U?.3 (-), U?.3 (-), U?.4 (GND), U?.4 (GND), U?.7 (REF1), U?.7 (REF1)
- net at Q?.14 (S2), Q?.5 (S2), Q?.6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: now also R?.1, U?.2 (+) (x2)
- net at Q?.14 (S2), Q?.5 (S2), Q?.6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: now also U?.2 (+)
- net +5V renamed VREF
- net VREF: now also U?.6 (REF2), U?.6 (REF2); no longer U?.5 (V+)
- net B renamed Curr_V
- net ~FAULT: no longer names the net of U?.17 (~FAULT)
- net ~FAULT: now also TP?.1
- new net Curr_U: U?.8
- new net Curr_W: U?.8
Other:
- note added: "INA240: REF1 and REF2 pins are swappable"
- moved on the sheet: C?, Q?, R?, U?

Commit message: micro-motor-v2: Schematic finished
Parts:
- C401: renamed from C?; footprint Capacitors_THT:CP_Radial_D4.0mm_P2.00mm -> Capacitor_THT:CP_Radial_D4.0mm_P2.00mm
- C402, C403, C406: renamed from C?; footprint Capacitors_SMD:C_0603 -> Capacitor_SMD:C_0402_1005Metric
- C404, C405: renamed from C?; footprint Capacitors_SMD:C_0603 -> Capacitor_SMD:C_0603_1608Metric
- Q401, Q402, Q403: renamed from Q?; footprint DFN-12-2EP_3.3x5mm_Pitch0.65mm:DFN-12-2EP_3.3x5mm_Pitch0.65mm -> FDMD82xx:DFN-12-2EP_3.3x5mm_Pitch0.65mm
- R401: renamed from R?; footprint (none) -> Resistor_SMD:R_0402_1005Metric
- R402, R403, R404: renamed from R?; footprint Resistors_SMD:R_0805 -> Resistor_SMD:R_0805_2012Metric
- TP401: renamed from TP?; footprint (none) -> TestPoint:TestPoint_Pad_D1.0mm
- U401: renamed from U?; footprint (none) -> Package_DFN_QFN:QFN-32-1EP_5x5mm_P0.5mm_EP3.45x3.45mm
- gave numbers to parts that had none: 3

Commit message: micro-motor-v2: layout: components placed
Connections:
- net Curr_U: now also U402.8; no longer U404.8
- net Curr_W: now also U404.8; no longer U402.8
- net OUT_U: now also Q401.10, Q401.11 (G1R), Q401.7, Q401.8, Q401.9; no longer Q403.10, Q403.11 (G1R), Q403.7, Q403.8, Q403.9
- net OUT_W: now also Q403.10, Q403.11 (G1R), Q403.7, Q403.8, Q403.9; no longer Q401.10, Q401.11 (G1R), Q401.7, Q401.8, Q401.9
- net at Q403.12 (G1): now also U401.13 (GHC); no longer U401.5 (GHA)
- net at Q403.14 (S2), Q403.5 (S2), Q403.6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: now also U401.16 (SLC); no longer U401.8 (SLA)
- net at Q403.4 (G2): now also U401.15 (GLC); no longer U401.7 (GLA)
- net at Q401.12 (G1): now also U401.5 (GHA); no longer U401.13 (GHC)
- net at Q401.14 (S2), Q401.5 (S2), Q401.6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: now also U401.8 (SLA); no longer U401.16 (SLC)
- net at Q401.4 (G2): now also U401.7 (GLA); no longer U401.15 (GLC)
Other:
- moved on the sheet: Q401, Q403, R402, R404, U402, U404
Changed lines of the file:
@@
-$EndComp
-$Comp
-L FDMD82xx:FDMD82xx Q403
-U 1 1 5A50285C
-P 9550 1500
-F 0 "Q403" H 9200 1400 50  0000 L CNN
-F 1 "FDMD82xx" H 9050 1500 50  0000 L CNN
-F 2 "FDMD82xx:DFN-12-2EP_3.3x5mm_Pitch0.65mm" H 9650 1550 60  0001 C CNN
-F 3 "" H 9500 1650 50  0001 L CNN
-	1    9550 1500
-	1    0    0    -1
 $EndComp
 $Comp
@@
 OUT_U
 $Comp
-L FDMD82xx:FDMD82xx Q401
-U 1 1 5A505C4C
-P 7300 3500
-F 0 "Q401" H 6950 3400 50  0000 L CNN
-F 1 "FDMD82xx" H 6800 3500 50  0000 L CNN
-F 2 "FDMD82xx:DFN-12-2EP_3.3x5mm_Pitch0.65mm" H 7400 3550 60  0001 C CNN
-F 3 "" H 7250 3650 50  0001 L CNN
-	1    7300 3500
-	1    0    0    -1
-$EndComp
-$Comp
 L power:+24V #PWR0410
 U 1 1 5A505C52
@@
 Text HLabel 7850 3500 2    60   Output ~ 0
 OUT_W
-$Comp
-L FDMD82xx:FDMD82xx Q402
-U 1 1 5A506004
-P 8450 2550
-F 0 "Q402" H 8100 2450 50  0000 L CNN
-F 1 "FDMD82xx" H 7950 2550 50  0000 L CNN
-F 2 "FDMD82xx:DFN-12-2EP_3.3x5mm_Pitch0.65mm" H 8550 2600 60  0001 C CNN
-F 3 "" H 8400 2700 50  0001 L CNN
-	1    8450 2550
-	1    0    0    -1
-$EndComp
 $Comp
 L power:+24V #PWR0413
@@
 	8000 5600 8000 5700
 $Comp
-L Device:R R404
-U 1 1 5D9F0A57
-P 9600 5300
-F 0 "R404" V 9680 5300 50  0000 C CNN
-F 1 "5m" V 9600 5300 50  0000 C CNN
-F 2 "Resistor_SMD:R_0805_2012Metric" V 9530 5300 50  0001 C CNN
-F 3 "" H 9600 5300 50  0001 C CNN
-	1    9600 5300
-	1    0    0    -1
-$EndComp
-$Comp
 L power:GND #PWR0417
 U 1 1 5D9F0A61
@@
 Wire Wire Line
 	9600 5450 9600 5550
-$Comp
-L Amplifier_Current:INA240A2PW U404
-U 1 1 5D9F0A6C
-P 9100 5300
-F 0 "U404" H 9100 5781 50  0000 C CNN
-F 1 "INA240A2PW" V 8850 5750 50  0000 C CNN
-F 2 "Package_SO:TSSOP-8_4.4x3mm_P0.65mm" H 9100 4650 50  0001 C CNN
-F 3 "http://www.ti.com/lit/ds/symlink/ina240.pdf" H 9250 5450 50  0001 C CNN
-	1    9100 5300
-	-1   0    0    -1
-$EndComp
 Wire Wire Line
 	8800 5300 8800 5250
@@
 Wire Wire Line
 	9100 5600 9100 5700
-$Comp
-L Device:R R402
-U 1 1 5D9FEF80
-P 7350 5300
-F 0 "R402" V 7430 5300 50  0000 C CNN
-F 1 "5m" V 7350 5300 50  0000 C CNN
-F 2 "Resistor_SMD:R_0805_2012Metric" V 7280 5300 50  0001 C CNN
-F 3 "" H 7350 5300 50  0001 C CNN
-	1    7350 5300
-	1    0    0    -1
-$EndComp
 $Comp
 L power:GND #PWR0411
@@
 Wire Wire Line
 	7350 5450 7350 5550
-$Comp
-L Amplifier_Current:INA240A2PW U402
-U 1 1 5D9FEF95
-P 6850 5300
-F 0 "U402" H 6850 5781 50  0000 C CNN
-F 1 "INA240A2PW" V 6600 5750 50  0000 C CNN
-F 2 "Package_SO:TSSOP-8_4.4x3mm_P0.65mm" H 6850 4650 50  0001 C CNN
-F 3 "http://www.ti.com/lit/ds/symlink/ina240.pdf" H 7000 5450 50  0001 C CNN
-	1    6850 5300
-	-1   0    0    -1
-$EndComp
 Text HLabel 6550 5250 1    50   Output ~ 0
 Curr_W
@@
 	1    0    0    -1
 $EndComp
+$Comp
+L Device:R R402
+U 1 1 5D9FEF80
+P 9600 5300
+F 0 "R402" V 9680 5300 50  0000 C CNN
+F 1 "5m" V 9600 5300 50  0000 C CNN
+F 2 "Resistor_SMD:R_0805_2012Metric" V 9530 5300 50  0001 C CNN
+F 3 "" H 9600 5300 50  0001 C CNN
+	1    9600 5300
+	1    0    0    -1
+$EndComp
+$Comp
+L Amplifier_Current:INA240A2PW U404
+U 1 1 5D9F0A6C
+P 6850 5300
+F 0 "U404" H 6850 5781 50  0000 C CNN
+F 1 "INA240A2PW" V 6600 5750 50  0000 C CNN
+F 2 "Package_SO:TSSOP-8_4.4x3mm_P0.65mm" H 6850 4650 50  0001 C CNN
+F 3 "http://www.ti.com/lit/ds/symlink/ina240.pdf" H 7000 5450 50  0001 C CNN
+	1    6850 5300
+	-1   0    0    -1
+$EndComp
+$Comp
+L Amplifier_Current:INA240A2PW U402
+U 1 1 5D9FEF95
+P 9100 5300
+F 0 "U402" H 9100 5781 50  0000 C CNN
+F 1 "INA240A2PW" V 8850 5750 50  0000 C CNN
+F 2 "Package_SO:TSSOP-8_4.4x3mm_P0.65mm" H 9100 4650 50  0001 C CNN
+F 3 "http://www.ti.com/lit/ds/symlink/ina240.pdf" H 9250 5450 50  0001 C CNN
+	1    9100 5300
+	-1   0    0    -1
+$EndComp
+$Comp
+L FDMD82xx:FDMD82xx Q403
+U 1 1 5A50285C
+P 7300 3500
+F 0 "Q403" H 6950 3400 50  0000 L CNN
+F 1 "FDMD82xx" H 6800 3500 50  0000 L CNN
+F 2 "FDMD82xx:DFN-12-2EP_3.3x5mm_Pitch0.65mm" H 7400 3550 60  0001 C CNN
+F 3 "" H 7250 3650 50  0001 L CNN
+	1    7300 3500
+	1    0    0    -1
+$EndComp
+$Comp
+L FDMD82xx:FDMD82xx Q402
+U 1 1 5A506004
+P 8450 2550
+F 0 "Q402" H 8100 2450 50  0000 L CNN
+F 1 "FDMD82xx" H 7950 2550 50  0000 L CNN
+F 2 "FDMD82xx:DFN-12-2EP_3.3x5mm_Pitch0.65mm" H 8550 2600 60  0001 C CNN
+F 3 "" H 8400 2700 50  0001 L CNN
+	1    8450 2550
+	1    0    0    -1
+$EndComp
+$Comp
+L FDMD82xx:FDMD82xx Q401
+U 1 1 5A505C4C
+P 9550 1500
+F 0 "Q401" H 9200 1400 50  0000 L CNN
+F 1 "FDMD82xx" H 9050 1500 50  0000 L CNN
+F 2 "FDMD82xx:DFN-12-2EP_3.3x5mm_Pitch0.65mm" H 9650 1550 60  0001 C CNN
+F 3 "" H 9500 1650 50  0001 L CNN
+	1    9550 1500
+	1    0    0    -1
+$EndComp
+$Comp
+L Device:R R404
+U 1 1 5D9F0A57
+P 7350 5300
+F 0 "R404" V 7430 5300 50  0000 C CNN
+F 1 "5m" V 7350 5300 50  0000 C CNN
+F 2 "Resistor_SMD:R_0805_2012Metric" V 7280 5300 50  0001 C CNN
+F 3 "" H 7350 5300 50  0001 C CNN
+	1    7350 5300
+	1    0    0    -1
+$EndComp

Commit message: micro-motor-v2: More capacitors, outline corners
Parts:
- added C407, C408, C409: 22µ 35V 1210, Capacitor_SMD:C_1210_3225Metric, symbol Device:C
- added C410, C411, C412: 100n, Capacitor_SMD:C_0402_1005Metric, symbol Device:C
- C401: footprint Capacitor_THT:CP_Radial_D4.0mm_P2.00mm -> Capacitor_THT:CP_Radial_D10.0mm_P5.00mm
- C402, C403: value 100n 50V -> 100n
Connections:
- net +24V: now also C407.1, C408.1, C409.1
- net +3V3: now also C410.1, C411.1, C412.1
- net GND: now also C407.2, C408.2, C409.2, C410.2, C411.2, C412.2
Other:
- note added: "DC-Link Capacitors\nPlace next to MOSFETs!"
- note added: "INA240 decoupling\ncapacitors"
- moved on the sheet: C403
Changed lines of the file:
@@
 P 2150 2400
 F 0 "C402" H 2175 2500 50  0000 L CNN
-F 1 "100n 50V" H 2175 2300 50  0000 L CNN
+F 1 "100n" H 2175 2300 50  0000 L CNN
 F 2 "Capacitor_SMD:C_0402_1005Metric" H 2188 2250 50  0001 C CNN
 F 3 "" H 2150 2400 50  0001 C CNN
@@
 F 0 "C401" H 1525 2500 50  0000 L CNN
 F 1 ">10µ 35V" H 1525 2300 50  0000 L CNN
-F 2 "Capacitor_THT:CP_Radial_D4.0mm_P2.00mm" H 1538 2250 50  0001 C CNN
+F 2 "Capacitor_THT:CP_Radial_D10.0mm_P5.00mm" H 1538 2250 50  0001 C CNN
 F 3 "" H 1500 2400 50  0001 C CNN
 	1    1500 2400
@@
 L Device:C C403
 U 1 1 5A78F36A
-P 2700 2400
-F 0 "C403" H 2725 2500 50  0000 L CNN
-F 1 "100n 50V" H 2725 2300 50  0000 L CNN
-F 2 "Capacitor_SMD:C_0402_1005Metric" H 2738 2250 50  0001 C CNN
-F 3 "" H 2700 2400 50  0001 C CNN
-	1    2700 2400
+P 2850 2400
+F 0 "C403" H 2875 2500 50  0000 L CNN
+F 1 "100n" H 2875 2300 50  0000 L CNN
+F 2 "Capacitor_SMD:C_0402_1005Metric" H 2888 2250 50  0001 C CNN
+F 3 "" H 2850 2400 50  0001 C CNN
+	1    2850 2400
 	1    0    0    -1
 $EndComp
@@
 L power:GND #PWR0404
 U 1 1 5A78F370
-P 2700 2650
-F 0 "#PWR0404" H 2700 2400 50  0001 C CNN
-F 1 "GND" H 2700 2500 50  0000 C CNN
-F 2 "" H 2700 2650 50  0001 C CNN
-F 3 "" H 2700 2650 50  0001 C CNN
-	1    2700 2650
-	1    0    0    -1
-$EndComp
-Wire Wire Line
-	2700 2650 2700 2550
-Wire Wire Line
-	2700 2250 2700 2150
-Connection ~ 2700 2150
+P 2850 2650
+F 0 "#PWR0404" H 2850 2400 50  0001 C CNN
+F 1 "GND" H 2850 2500 50  0000 C CNN
+F 2 "" H 2850 2650 50  0001 C CNN
+F 3 "" H 2850 2650 50  0001 C CNN
+	1    2850 2650
+	1    0    0    -1
+$EndComp
+Wire Wire Line
+	2850 2650 2850 2550
+Wire Wire Line
+	2850 2250 2850 2150
+Connection ~ 2850 2150
 Wire Wire Line
 	3750 2150 4550 2150
 Wire Wire Line
-	2150 2150 2700 2150
+	2150 2150 2850 2150
 Wire Wire Line
 	1500 2150 2150 2150
@@
 	3600 2650 4550 2650
 Wire Wire Line
-	2700 2150 3750 2150
+	2850 2150 3750 2150
 $Comp
 L Device:R R401
@@
 	1    0    0    -1
 $EndComp
+$Comp
+L Device:C C408
+U 1 1 5D8AC87D
+P 1850 6700
+F 0 "C408" H 1875 6800 50  0000 L CNN
+F 1 "22µ 35V 1210" H 1875 6600 50  0000 L CNN
+F 2 "Capacitor_SMD:C_1210_3225Metric" H 1888 6550 50  0001 C CNN
+F 3 "" H 1850 6700 50  0001 C CNN
+	1    1850 6700
+	1    0    0    -1
+$EndComp
+$Comp
+L Device:C C407
+U 1 1 5D8CF06D
+P 950 6700
+F 0 "C407" H 975 6800 50  0000 L CNN
+F 1 "22µ 35V 1210" H 975 6600 50  0000 L CNN
+F 2 "Capacitor_SMD:C_1210_3225Metric" H 988 6550 50  0001 C CNN
+F 3 "" H 950 6700 50  0001 C CNN
+	1    950  6700
+	1    0    0    -1
+$EndComp
+$Comp
+L Device:C C409
+U 1 1 5D8CF35F
+P 2750 6700
+F 0 "C409" H 2775 6800 50  0000 L CNN
+F 1 "22µ 35V 1210" H 2775 6600 50  0000 L CNN
+F 2 "Capacitor_SMD:C_1210_3225Metric" H 2788 6550 50  0001 C CNN
+F 3 "" H 2750 6700 50  0001 C CNN
+	1    2750 6700
+	1    0    0    -1
+$EndComp
+Wire Wire Line
+	950  6550 950  6450
+Wire Wire Line
+	950  6450 1850 6450
+Wire Wire Line
+	2750 6450 2750 6550
+Wire Wire Line
+	1850 6550 1850 6450
+Connection ~ 1850 6450
+Wire Wire Line
+	1850 6450 2750 6450
+Wire Wire Line
+	1850 6450 1850 6350
+Wire Wire Line
+	950  6850 950  6950
+Wire Wire Line
+	950  6950 1850 6950
+Wire Wire Line
+	2750 6950 2750 6850
+Wire Wire Line
+	1850 6850 1850 6950
+Connection ~ 1850 6950
+Wire Wire Line
+	1850 6950 2750 6950
+Wire Wire Line
+	1850 6950 1850 7050
+$Comp
+L power:GND #PWR0419
+U 1 1 5D9290AD
+P 1850 7050
+F 0 "#PWR0419" H 1850 6800 50  0001 C CNN
+F 1 "GND" H 1855 6877 50  0000 C CNN
+F 2 "" H 1850 7050 50  0001 C CNN
+F 3 "" H 1850 7050 50  0001 C CNN
+	1    1850 7050
+	1    0    0    -1
+$EndComp
+$Comp
+L power:+24V #PWR0418
+U 1 1 5D9294AA
+P 1850 6350
+F 0 "#PWR0418" H 1850 6200 50  0001 C CNN
+F 1 "+24V" H 1865 6523 50  0000 C CNN
+F 2 "" H 1850 6350 50  0001 C CNN
+F 3 "" H 1850 6350 50  0001 C CNN
+	1    1850 6350
+	1    0    0    -1
+$EndComp
+Text Notes 2200 6300 0    50   ~ 0
+DC-Link Capacitors\nPlace next to MOSFETs!
+$Comp
+L Device:C C410
+U 1 1 5D9BCA0F
+P 4550 6650
+F 0 "C410" H 4575 6750 50  0000 L CNN
+F 1 "100n" H 4575 6550 50  0000 L CNN
+F 2 "Capacitor_SMD:C_0402_1005Metric" H 4588 6500 50  0001 C CNN
+F 3 "" H 4550 6650 50  0001 C CNN
+	1    4550 6650
+	1    0    0    -1
+$EndComp
+$Comp
+L Device:C C411
+U 1 1 5D9BE679
+P 5000 6650
+F 0 "C411" H 5025 6750 50  0000 L CNN
+F 1 "100n" H 5025 6550 50  0000 L CNN
+F 2 "Capacitor_SMD:C_0402_1005Metric" H 5038 6500 50  0001 C CNN
+F 3 "" H 5000 6650 50  0001 C CNN
+	1    5000 6650
+	1    0    0    -1
+$EndComp
+$Comp
+L Device:C C412
+U 1 1 5D9BE947
+P 5500 6650
+F 0 "C412" H 5525 6750 50  0000 L CNN
+F 1 "100n" H 5525 6550 50  0000 L CNN
+F 2 "Capacitor_SMD:C_0402_1005Metric" H 5538 6500 50  0001 C CNN
+F 3 "" H 5500 6650 50  0001 C CNN
+	1    5500 6650
+	1    0    0    -1
+$EndComp
+Wire Wire Line
+	4550 6500 4550 6400
+Wire Wire Line
+	4550 6400 5000 6400
+Wire Wire Line
+	5500 6400 5500 6500
+Wire Wire Line
+	5500 6800 5500 6900
+Wire Wire Line
+	5500 6900 5000 6900
+Wire Wire Line
+	4550 6900 4550 6800
+Wire Wire Line
+	5000 6800 5000 6900
+Connection ~ 5000 6900
+Wire Wire Line
+	5000 6900 4550 6900
+Wire Wire Line
+	5000 6500 5000 6400
+Connection ~ 5000 6400
+Wire Wire Line
+	5000 6400 5500 6400
+Wire Wire Line
+	5000 6400 5000 6300
+Wire Wire Line
+	5000 6900 5000 7000
+Text Notes 5150 6300 0    50   ~ 0
+INA240 decoupling\ncapacitors
+$Comp
+L power:GND #PWR0421
+U 1 1 5DA17519
+P 5000 7000
+F 0 "#PWR0421" H 5000 6750 50  0001 C CNN
+F 1 "GND" H 5005 6827 50  0000 C CNN
+F 2 "" H 5000 7000 50  0001 C CNN
+F 3 "" H 5000 7000 50  0001 C CNN
+	1    5000 7000
+	1    0    0    -1
+$EndComp
+$Comp
+L power:+3V3 #PWR0420
+U 1 1 5DA17E14
+P 5000 6300
+F 0 "#PWR0420" H 5000 6150 50  0001 C CNN
+F 1 "+3V3" H 5015 6473 50  0000 C CNN
+F 2 "" H 5000 6300 50  0001 C CNN
+F 3 "" H 5000 6300 50  0001 C CNN
+	1    5000 6300
+	1    0    0    -1
+$EndComp

Commit message: micro-motor-v2: Layout...
Connections:
- net GND: no longer C401.2, C402.2, C403.2, C404.2, C407.2, C408.2, C409.2, R402.2, R403.2, R404.2, U401.23 (AGND), U401.31 (PGND), U401.33 (GND), U402.3 (-), U403.3 (-), U404.3 (-)
- net GND_C: now reaches Q403.14 (S2), Q403.5 (S2), Q403.6, R404.1, U401.16 (SLC), U404.2 (+)
- net GND_A: now reaches Q401.14 (S2), Q401.5 (S2), Q401.6, R402.1, U401.8 (SLA), U402.2 (+)
- net GND_B: now reaches Q402.14 (S2), Q402.5 (S2), Q402.6, R403.1, U401.9 (SLB), U403.2 (+)
- new net GNDPWR: C401.2, C402.2, C403.2, C404.2, C407.2, C408.2, C409.2, R402.2, R403.2, R404.2, U401.23 (AGND), U401.31 (PGND), U401.33 (GND), U402.3 (-), U403.3 (-), U404.3 (-)
Changed lines of the file:
@@
-$EndComp
-$Comp
-L power:GND #PWR0402
-U 1 1 5A4FE4D1
-P 1500 2650
-F 0 "#PWR0402" H 1500 2400 50  0001 C CNN
-F 1 "GND" H 1500 2500 50  0000 C CNN
-F 2 "" H 1500 2650 50  0001 C CNN
-F 3 "" H 1500 2650 50  0001 C CNN
-	1    1500 2650
-	1    0    0    -1
-$EndComp
-$Comp
-L power:GND #PWR0403
-U 1 1 5A4FE4F8
-P 2150 2650
-F 0 "#PWR0403" H 2150 2400 50  0001 C CNN
-F 1 "GND" H 2150 2500 50  0000 C CNN
-F 2 "" H 2150 2650 50  0001 C CNN
-F 3 "" H 2150 2650 50  0001 C CNN
-	1    2150 2650
-	1    0    0    -1
 $EndComp
 $Comp
@@
 	1    0    0    -1
 $EndComp
-$Comp
-L power:GND #PWR0406
-U 1 1 5A4FE87C
-P 3600 3250
-F 0 "#PWR0406" H 3600 3000 50  0001 C CNN
-F 1 "GND" H 3600 3100 50  0000 C CNN
-F 2 "" H 3600 3250 50  0001 C CNN
-F 3 "" H 3600 3250 50  0001 C CNN
-	1    3600 3250
-	1    0    0    -1
-$EndComp
 Text HLabel 4350 3850 0    60   Input ~ 0
 MOSI
@@
 ~CS
 $Comp
-L power:GND #PWR0407
-U 1 1 5A4FF46D
-P 5350 4700
-F 0 "#PWR0407" H 5350 4450 50  0001 C CNN
-F 1 "GND" H 5350 4550 50  0000 C CNN
-F 2 "" H 5350 4700 50  0001 C CNN
-F 3 "" H 5350 4700 50  0001 C CNN
-	1    5350 4700
-	1    0    0    -1
-$EndComp
-$Comp
 L power:+24V #PWR0416
 U 1 1 5A502CAF
@@
 F 3 "" H 2850 2400 50  0001 C CNN
 	1    2850 2400
-	1    0    0    -1
-$EndComp
-$Comp
-L power:GND #PWR0404
-U 1 1 5A78F370
-P 2850 2650
-F 0 "#PWR0404" H 2850 2400 50  0001 C CNN
-F 1 "GND" H 2850 2500 50  0000 C CNN
-F 2 "" H 2850 2650 50  0001 C CNN
-F 3 "" H 2850 2650 50  0001 C CNN
-	1    2850 2650
 	1    0    0    -1
 $EndComp
@@
 Wire Wire Line
 	5350 4450 5350 4700
-$Comp
-L power:GND #PWR0414
-U 1 1 5DE98D31
-P 8500 5900
-F 0 "#PWR0414" H 8500 5650 50  0001 C CNN
-F 1 "GND" H 8505 5727 50  0000 C CNN
-F 2 "" H 8500 5900 50  0001 C CNN
-F 3 "" H 8500 5900 50  0001 C CNN
-	1    8500 5900
-	1    0    0    -1
-$EndComp
 Wire Wire Line
 	8500 5450 8500 5550
@@
 Wire Wire Line
 	8100 5800 8100 5600
-Connection ~ 8100 5800
-Wire Wire Line
-	8100 5800 8500 5800
-Connection ~ 8500 5800
-Wire Wire Line
-	8500 5800 8500 5900
 $Comp
 L drv8323s:DRV8320S U401
@@
 Connection ~ 8500 5550
 Wire Wire Line
-	8500 5550 8500 5800
-Wire Wire Line
 	8300 5200 8400 5200
 Wire Wire Line
@@
 Wire Wire Line
 	8000 5600 8000 5700
-$Comp
-L power:GND #PWR0417
-U 1 1 5D9F0A61
-P 9600 5900
-F 0 "#PWR0417" H 9600 5650 50  0001 C CNN
-F 1 "GND" H 9605 5727 50  0000 C CNN
-F 2 "" H 9600 5900 50  0001 C CNN
-F 3 "" H 9600 5900 50  0001 C CNN
-	1    9600 5900
-	1    0    0    -1
-$EndComp
 Wire Wire Line
 	9600 5450 9600 5550
@@
 Wire Wire Line
 	9000 5800 9200 5800
-Connection ~ 9200 5800
-Wire Wire Line
-	9200 5800 9600 5800
-Connection ~ 9600 5800
-Wire Wire Line
-	9600 5800 9600 5900
 Wire Wire Line
 	9400 5400 9500 5400
@@
 Connection ~ 9600 5550
 Wire Wire Line
-	9600 5550 9600 5800
-Wire Wire Line
 	9400 5200 9500 5200
 Wire Wire Line
@@
 Wire Wire Line
 	9100 5600 9100 5700
-$Comp
-L power:GND #PWR0411
-U 1 1 5D9FEF8A
-P 7350 5900
-F 0 "#PWR0411" H 7350 5650 50  0001 C CNN
-F 1 "GND" H 7355 5727 50  0000 C CNN
-F 2 "" H 7350 5900 50  0001 C CNN
-F 3 "" H 7350 5900 50  0001 C CNN
-	1    7350 5900
-	1    0    0    -1
-$EndComp
 Wire Wire Line
 	7350 5450 7350 5550
@@
 Wire Wire Line
 	6950 5800 6950 5600
-Connection ~ 6950 5800
-Wire Wire Line
-	6950 5800 7350 5800
-Connection ~ 7350 5800
-Wire Wire Line
-	7350 5800 7350 5900
 Wire Wire Line
 	7150 5400 7250 5400
@@
 	7250 5550 7350 5550
 Connection ~ 7350 5550
-Wire Wire Line
-	7350 5550 7350 5800
 Wire Wire Line
 	7150 5200 7250 5200
@@
 	1850 6950 1850 7050
 $Comp
-L power:GND #PWR0419
-U 1 1 5D9290AD
-P 1850 7050
-F 0 "#PWR0419" H 1850 6800 50  0001 C CNN
-F 1 "GND" H 1855 6877 50  0000 C CNN
-F 2 "" H 1850 7050 50  0001 C CNN
-F 3 "" H 1850 7050 50  0001 C CNN
-	1    1850 7050
-	1    0    0    -1
-$EndComp
-$Comp
 L power:+24V #PWR0418
 U 1 1 5D9294AA
@@
 	1    0    0    -1
 $EndComp
+Text Label 7350 4750 0    50   ~ 0
+GND_C
+Text Label 8500 4550 0    50   ~ 0
+GND_B
+Text Label 9600 4550 0    50   ~ 0
+GND_A
+$Comp
+L power:GNDPWR #PWR0121
+U 1 1 5D8FA43B
+P 9600 5900
+F 0 "#PWR0121" H 9600 5700 50  0001 C CNN
+F 1 "GNDPWR" H 9604 5746 50  0000 C CNN
+F 2 "" H 9600 5850 50  0001 C CNN
+F 3 "" H 9600 5850 50  0001 C CNN
+	1    9600 5900
+	1    0    0    -1
+$EndComp
+$Comp
+L power:GNDPWR #PWR0122
+U 1 1 5D8FA873
+P 8500 5900
+F 0 "#PWR0122" H 8500 5700 50  0001 C CNN
+F 1 "GNDPWR" H 8504 5746 50  0000 C CNN
+F 2 "" H 8500 5850 50  0001 C CNN
+F 3 "" H 8500 5850 50  0001 C CNN
+	1    8500 5900
+	1    0    0    -1
+$EndComp
+$Comp
+L power:GNDPWR #PWR0123
+U 1 1 5D8FADA6
+P 7350 5900
+F 0 "#PWR0123" H 7350 5700 50  0001 C CNN
+F 1 "GNDPWR" H 7354 5746 50  0000 C CNN
+F 2 "" H 7350 5850 50  0001 C CNN
+F 3 "" H 7350 5850 50  0001 C CNN
+	1    7350 5900
+	1    0    0    -1
+$EndComp
+Wire Wire Line
+	7350 5550 7350 5900
+Wire Wire Line
+	8500 5550 8500 5900
+Wire Wire Line
+	9600 5550 9600 5900
+$Comp
+L power:GND #PWR0124
+U 1 1 5D8FCDAB
+P 9200 5900
+F 0 "#PWR0124" H 9200 5650 50  0001 C CNN
+F 1 "GND" H 9205 5727 50  0000 C CNN
+F 2 "" H 9200 5900 50  0001 C CNN
+F 3 "" H 9200 5900 50  0001 C CNN
+	1    9200 5900
+	1    0    0    -1
+$EndComp
+Wire Wire Line
+	9200 5900 9200 5800
+Connection ~ 9200 5800
+Wire Wire Line
+	8100 5800 8100 5900
+Connection ~ 8100 5800
+Wire Wire Line
+	6950 5800 6950 5900
+Connection ~ 6950 5800
+$Comp
+L power:GND #PWR0125
+U 1 1 5D92A2AB
+P 8100 5900
+F 0 "#PWR0125" H 8100 5650 50  0001 C CNN
+F 1 "GND" H 8105 5727 50  0000 C CNN
+F 2 "" H 8100 5900 50  0001 C CNN
+F 3 "" H 8100 5900 50  0001 C CNN
+	1    8100 5900
+	1    0    0    -1
+$EndComp
+$Comp
+L power:GND #PWR0126
+U 1 1 5D92A5A1
+P 6950 5900
+F 0 "#PWR0126" H 6950 5650 50  0001 C CNN
+F 1 "GND" H 6955 5727 50  0000 C CNN
+F 2 "" H 6950 5900 50  0001 C CNN
+F 3 "" H 6950 5900 50  0001 C CNN
+	1    6950 5900
+	1    0    0    -1
+$EndComp
+$Comp
+L power:GNDPWR #PWR0127
+U 1 1 5D92E77E
+P 1850 7050
+F 0 "#PWR0127" H 1850 6850 50  0001 C CNN
+F 1 "GNDPWR" H 1854 6896 50  0000 C CNN
+F 2 "" H 1850 7000 50  0001 C CNN
+F 3 "" H 1850 7000 50  0001 C CNN
+	1    1850 7050
+	1    0    0    -1
+$EndComp
+$Comp
+L power:GNDPWR #PWR0128
+U 1 1 5D9342D5
+P 5350 4700
+F 0 "#PWR0128" H 5350 4500 50  0001 C CNN
+F 1 "GNDPWR" H 5354 4546 50  0000 C CNN
+F 2 "" H 5350 4650 50  0001 C CNN
+F 3 "" H 5350 4650 50  0001 C CNN
+	1    5350 4700
+	1    0    0    -1
+$EndComp
+$Comp
+L power:GNDPWR #PWR0129
+U 1 1 5D948CCD
+P 3600 3250
+F 0 "#PWR0129" H 3600 3050 50  0001 C CNN
+F 1 "GNDPWR" H 3604 3096 50  0000 C CNN
+F 2 "" H 3600 3200 50  0001 C CNN
+F 3 "" H 3600 3200 50  0001 C CNN
+	1    3600 3250
+	1    0    0    -1
+$EndComp
+$Comp
+L power:GNDPWR #PWR0130
+U 1 1 5D949560
+P 2150 2650
+F 0 "#PWR0130" H 2150 2450 50  0001 C CNN
+F 1 "GNDPWR" H 2154 2496 50  0000 C CNN
+F 2 "" H 2150 2600 50  0001 C CNN
+F 3 "" H 2150 2600 50  0001 C CNN
+	1    2150 2650
+	1    0    0    -1
+$EndComp
+$Comp
+L power:GNDPWR #PWR0131
+U 1 1 5D949F7C
+P 1500 2650
+F 0 "#PWR0131" H 1500 2450 50  0001 C CNN
+F 1 "GNDPWR" H 1504 2496 50  0000 C CNN
+F 2 "" H 1500 2600 50  0001 C CNN
+F 3 "" H 1500 2600 50  0001 C CNN
+	1    1500 2650
+	1    0    0    -1
+$EndComp
+$Comp
+L power:GNDPWR #PWR0132
+U 1 1 5D94ADBC
+P 2850 2650
+F 0 "#PWR0132" H 2850 2450 50  0001 C CNN
+F 1 "GNDPWR" H 2854 2496 50  0000 C CNN
+F 2 "" H 2850 2600 50  0001 C CNN
+F 3 "" H 2850 2600 50  0001 C CNN
+	1    2850 2650
+	1    0    0    -1
+$EndComp
