File: kicad/micro-motor-v2.2/Motordriver.kicad_sch (KiCad schematic)
At the start: 23 parts, among them Q401 FDMD82xx, Q402 FDMD82xx, Q403 FDMD82xx, U401 DRV8320S, U402 INA240A2PW, U403 INA240A2PW, U404 INA240A2PW

Commit message: ready to order
Other:
- title: Micro-Motor V2.1 -> Micro-Motor V2.2
Changed lines of the file:
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@@
   (paper "A4")
   (title_block
-    (title "Micro-Motor V2.1")
+    (title "Micro-Motor V2.2")
     (date "2021-07-31")
     (rev "1")
