File: kicad/micro-motor-v2.2/Power_Supply.kicad_sch (KiCad schematic)
At the start: 6 parts, among them U501 LMZM23601V3, U502 LMZM23601V5

Commit message: ready to order
Other:
- title: Micro-Motor V2.1 -> Micro-Motor V2.2
Changed lines of the file:
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@@
   (paper "A4")
   (title_block
-    (title "Micro-Motor V2.1")
+    (title "Micro-Motor V2.2")
     (date "2021-07-31")
     (rev "1")
